File: hardware/iasis/controller-sense.kicad_sch (KiCad schematic)
At the start: 28 parts, among them U1141 TMUX1511PWR, U1142 TMUX1511PWR

Commit message: Add the CM5 carrier design for reference
The first board revision: a Raspberry Pi CM5 carrier with M.2 NVMe,
Ethernet and five USB 3 and USB-PD ports, as it stood before the compact
hub replaced it, squashed from 45 commits.
Parts:
- C1141, C1147: LCSC C1525 -> (none); MPN CL05B104KO5NNNC -> (none); Manufacturer Samsung Electro-Mechanics -> (none)
- C1142, C1143, C1144, C1145, C1146, C1148: LCSC C15195 -> (none); MPN CL05B103KB5NNNC -> (none); Manufacturer Samsung Electro-Mechanics -> (none)
- R1141, R1144, R1147, R1150, R1153, R1156: LCSC C852949 -> (none); MPN RT0402BRD0790K9L -> (none); Manufacturer YAGEO -> (none)
- R1142, R1145, R1148, R1151, R1154, R1157: LCSC C2991528 -> (none); MPN THC02H1002BT -> (none); Manufacturer FH (Guangdong Fenghua Advanced Tech) -> (none)
- R1143, R1146, R1149, R1152, R1155, R1158: LCSC C5122071 -> (none); MPN ARG02BTC4702 -> (none); Manufacturer Viking Tech -> (none)
- U1141, U1142: LCSC C2866750 -> (none); MPN TMUX1511PWR -> (none); Manufacturer Texas Instruments -> (none)
Connections:
- net HV_CHARGE renamed 24V_SYS
Other:
- note added: "VBUS = ADC voltage × 12.024 nominal; calibrate against measured rail voltage. VSYS_SENSE reads 24V_SYS on the same scale. The switches are open during reset or loss of 3V3_AON. The 47k resistors limit power-off ADC voltage from switch leakage."
- note removed: "VBUS = ADC voltage × 12.024 nominal; calibrate against measured rail voltage. VSYS_SENSE reads HV_CHARGE_SYS on the same scale. The switches are open during reset or loss of 3V3_AON. The 47k resistors limit power-off ADC voltage from switch leakage."
