File: hardware/iasis/controller-temperature.kicad_sch (KiCad schematic)
At the start: 6 parts

Commit message: Add the CM5 carrier design for reference
The first board revision: a Raspberry Pi CM5 carrier with M.2 NVMe,
Ethernet and five USB 3 and USB-PD ports, as it stood before the compact
hub replaced it, squashed from 45 commits.
Parts:
- C1191, C1192: LCSC C15195 -> (none); MPN CL05B103KB5NNNC -> (none); Manufacturer Samsung Electro-Mechanics -> (none)
- R1191, R1192: LCSC C25744 -> (none); MPN 0402WGF1002TCE -> (none); Manufacturer UNI-ROYAL(Uniroyal Elec) -> (none)
- TH1191, TH1192: LCSC C440252 -> (none); Manufacturer Murata Electronics -> (none)
