File: hardware/iasis/hub.kicad_sch (KiCad schematic)
At the start: 57 parts, among them U201 USB7206CT/KDX, U204 SN74AUP1G08DCKR, Y201 X322525MSB4SI

Commit message: Add the CM5 carrier design for reference
The first board revision: a Raspberry Pi CM5 carrier with M.2 NVMe,
Ethernet and five USB 3 and USB-PD ports, as it stood before the compact
hub replaced it, squashed from 45 commits.
Parts:
- added C224, C225: 100n, Capacitor_SMD:C_0402_1005Metric, symbol Device:C
- added U202: HD3SS3212IRKSR, Package_DFN_QFN:DHVQFN-20-1EP_2.5x4.5mm_P0.5mm_EP1x3mm, symbol Iasis:HD3SS3212IRKSR
- added U203: TMUX1511PWR, Package_SO:TSSOP-14_4.4x5mm_P0.65mm, symbol Iasis:TMUX1511PWR
- C201, C202: LCSC C1562 -> (none); MPN 0402CG330J500NT -> (none); Manufacturer FH (Guangdong Fenghua Advanced Tech) -> (none)
- C203, C204, C205, C206, C207, C208, C209, C210, C212, C213, C214, C215, C216, C217, C218, C219, C220, C222, C223, C226: LCSC C1525 -> (none); MPN CL05B104KO5NNNC -> (none); Manufacturer Samsung Electro-Mechanics -> (none)
- C211, C221: LCSC C19702 -> (none); MPN CL10A106KP8NNNC -> (none); Manufacturer Samsung Electro-Mechanics -> (none)
- R201: LCSC C25752 -> (none); MPN 0402WGF1202TCE -> (none); Manufacturer UNI-ROYAL(Uniroyal Elec) -> (none)
- R202, R207, R208, R209, R210, R211, R212, R213, R214, R215: LCSC C25744 -> (none); MPN 0402WGF1002TCE -> (none); Manufacturer UNI-ROYAL(Uniroyal Elec) -> (none)
- R203, R204, R205, R206: LCSC C25764 -> (none); MPN 0402WGF2003TCE -> (none); Manufacturer UNI-ROYAL(Uniroyal Elec) -> (none)
- R216: value 49.9k 1% -> 100k; LCSC C25897 -> (none); MPN 0402WGF4992TCE -> (none); Manufacturer UNI-ROYAL(Uniroyal Elec) -> (none)
- R217, R218, R219, R220, R221, R222, R223, R224, R225, R226, R227, R228, R229, R230: LCSC C25741 -> (none); MPN 0402WGF1003TCE -> (none); Manufacturer UNI-ROYAL(Uniroyal Elec) -> (none)
- U201: Manufacturer Microchip Tech -> Microchip
- U204: Manufacturer Texas Instruments -> (none)
- Y201: Manufacturer YXC Crystal Oscillators -> YXC
Connections:
- net 3V3_AON: now also C224.1, C225.1, U202.6 (VCC), U203.14 (VDD)
- net EXT_D_N: now also U203.12 (S4); no longer U201.90 (USB2UP_DM)
- net EXT_D_P: now also U203.9 (S3); no longer U201.89 (USB2UP_DP)
- net EXT_RX_N: now also U202.12 (C1N); no longer U201.95 (USB3UP_RXDM)
- net EXT_RX_P: now also U202.13 (C1P); no longer U201.94 (USB3UP_RXDP)
- net EXT_TX_N: now also U202.14 (C0N); no longer C223.2
- net EXT_TX_P: now also U202.15 (C0P); no longer C222.2
- net GND: now also C224.2, C225.2, U202.11 (GND), U202.2 (OE_N), U202.20 (GND), U202.21 (EP), U202.5 (GND), U203.7 (GND)
- net VCORE renamed 1V1_HUB
- new net CM5_USB3A_D_N: U203.5 (S2)
- new net CM5_USB3A_D_P: U203.2 (S1)
- new net CM5_USB3A_RX_N: U202.18 (B0N)
- new net CM5_USB3A_RX_P: U202.19 (B0P)
- new net CM5_USB3A_TX_N: U202.16 (B1N)
- new net CM5_USB3A_TX_P: U202.17 (B1P)
- new net MUX_RX_N: U201.94 (USB3UP_RXDP), U202.8 (A1N)
- new net MUX_RX_P: U201.95 (USB3UP_RXDM), U202.7 (A1P)
- new net MUX_TX_N: C223.2, U202.4 (A0N)
- new net MUX_TX_P: C222.2, U202.3 (A0P)
- new net SEL_CM5: U203.1 (SEL1), U203.4 (SEL2)
- new net SEL_EXT: U202.9 (SEL), U203.10 (SEL3), U203.13 (SEL4)
- new net UP_D_N: U201.90 (USB2UP_DM), U203.11 (D4), U203.6 (D2)
- new net UP_D_P: U201.89 (USB2UP_DP), U203.3 (D1), U203.8 (D3)
- no-connect marks 11 -> 13
Other:
- note added: "Configuration 3: CFG_STRAP1 10k, CFG_STRAP2/3 200k pull-downs. CFG_NON_REM and CFG_BC_EN 200k pull-downs: all ports removable, no battery charging. Boots from internal ROM; no SPI flash or OTP setup. PF26/PF27 are the SMBus client on TCA9548 channel 6 (HUB_SCL/HUB_SDA, 100k pull-downs). With HUB_SMB_EN off they read low at reset and the hub attaches on its own; firmware powers the pull-ups and pu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"
- note removed: "Configuration 3: CFG_STRAP1 10k; CFG_STRAP2/3, NON_REM and BC_EN 200k pull-downs. Internal ROM boot; all ports removable; battery charging detection off. HUB_SCL/SDA stay low during reset for autonomous attachment. RESET_N = AON_RESET_N AND HUB_RUN; HUB_RUN has a pull-up. The external host reaches the hub directly through the upstream orientation mux. HUB_UP_VBUS is a hardware divider from host V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"
