File: hardware/iasis/hub.kicad_sch (KiCad schematic)
At the start: 57 parts, among them U201 USB7206CT/KDX, U204 SN74AUP1G08DCKR, Y201 X322525MSB4SI

Commit message: fix: correct core power and recovery circuitry
Parts:
- R216: value 49.9k 1% -> 10k; LCSC C137969 -> C25744; MPN RC0402FR-0749K9L -> 0402WGF1002TCE; Manufacturer YAGEO -> UNI-ROYAL(Uniroyal Elec)
Connections:
- net 3V3_AON: now also R216.2
- net GND: no longer R216.2
Other:
- note added: "Configuration 3: CFG_STRAP1 10k; CFG_STRAP2/3, NON_REM and BC_EN 200k pull-downs. Internal ROM boot; all ports removable; battery charging detection off. HUB_SCL/SDA stay low during reset for autonomous attachment. RESET_N = AON_RESET_N AND HUB_RUN; HUB_RUN has a pull-up. The external host reaches the hub directly through the upstream orientation mux. HUB_UP_VBUS has a 10k pull-up to 3V3_AON and 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"
- note removed: "Configuration 3: CFG_STRAP1 10k; CFG_STRAP2/3, NON_REM and BC_EN 200k pull-downs. Internal ROM boot; all ports removable; battery charging detection off. HUB_SCL/SDA stay low during reset for autonomous attachment. RESET_N = AON_RESET_N AND HUB_RUN; HUB_RUN has a pull-up. The external host reaches the hub directly through the upstream orientation mux. HUB_UP_VBUS is a hardware divider from host V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"
- moved on the sheet: R216
Changed lines of the file:
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@@
 		)
 	)
-	(text "Configuration 3: CFG_STRAP1 10k; CFG_STRAP2/3, NON_REM and BC_EN 200k pull-downs.\nInternal ROM boot; all ports removable; battery charging detection off.\nHUB_SCL/SDA stay low during reset for autonomous attachment.\nRESET_N = AON_RESET_N AND HUB_RUN; HUB_RUN has a pull-up.\nThe external host reaches the hub directly through the upstream orientation mux.\nHUB_UP_VBUS is a hardware divider from host VBUS; MCU firmware is not needed to enumerate.\nPort 6 USB2 connects the RP2354. Target power is controlled independently of PRT_CTL1-6.\nUpstream TX uses C222/C223; downstream TX coupling is on the repeated port sheets.\nSuperSpeed lanes support native rate negotiation; USB2 D+/D- are never polarity swapped."
+	(text "Configuration 3: CFG_STRAP1 10k; CFG_STRAP2/3, NON_REM and BC_EN 200k pull-downs.\nInternal ROM boot; all ports removable; battery charging detection off.\nHUB_SCL/SDA stay low during reset for autonomous attachment.\nRESET_N = AON_RESET_N AND HUB_RUN; HUB_RUN has a pull-up.\nThe external host reaches the hub directly through the upstream orientation mux.\nHUB_UP_VBUS has a 10k pull-up to 3V3_AON and follows hub power; MCU firmware is not needed to enumerate.\nPort 6 USB2 connects the RP2354. Target power is controlled independently of PRT_CTL1-6.\nUpstream TX uses C222/C223; downstream TX coupling is on the repeated port sheets.\nSuperSpeed lanes support native rate negotiation; USB2 D+/D- are never polarity swapped."
 		(exclude_from_sim no)
 		(at 287.02 172.72 0)
@@
 	)
 	(junction
-		(at 38.1 210.82)
-		(diameter 0)
-		(color 0 0 0 0)
-	)
-	(junction
 		(at 287.02 55.88)
 		(diameter 0)
@@
 	(wire
 		(pts
-			(xy 38.1 203.2) (xy 38.1 200.66)
-		)
-		(stroke
-			(width 0)
-			(type default)
-		)
-	)
-	(wire
-		(pts
 			(xy 205.74 55.88) (xy 208.28 55.88)
 		)
@@
 	(wire
 		(pts
-			(xy 33.02 210.82) (xy 38.1 210.82)
-		)
-		(stroke
-			(width 0)
-			(type default)
-		)
-	)
-	(wire
-		(pts
-			(xy 38.1 210.82) (xy 55.88 210.82)
+			(xy 33.02 210.82) (xy 55.88 210.82)
 		)
 		(stroke
@@
 		)
 	)
+	(global_label "3V3_AON"
+		(shape input)
+		(at 38.1 208.28 0)
+		(effects
+			(font
+				(size 1.27 1.27)
+			)
+			(justify left)
+		)
+		(property "Intersheetrefs" "${INTERSHEET_REFS}"
+			(at 38.1 208.28 0)
+			(hide yes)
+			(show_name no)
+			(do_not_autoplace no)
+			(effects
+				(font
+					(size 1.27 1.27)
+				)
+			)
+		)
+	)
 	(global_label "HUB_SDA"
 		(shape input)
@@
 	(symbol
 		(lib_id "Device:R")
-		(at 38.1 207.01 0)
+		(at 38.1 204.47 0)
 		(unit 1)
 		(body_style 1)
@@
 		(dnp no)
 		(property "Reference" "R216"
-			(at 40.64 205.74 0)
+			(at 40.64 203.2 0)
 			(show_name no)
 			(do_not_autoplace no)
@@
 			)
 		)
-		(property "Value" "49.9k 1%"
-			(at 40.64 208.28 0)
+		(property "Value" "10k"
+			(at 40.64 205.74 0)
 			(show_name no)
 			(do_not_autoplace no)
@@
 		)
 		(property "Footprint" "Resistor_SMD:R_0402_1005Metric"
-			(at 38.1 207.01 0)
+			(at 38.1 204.47 0)
 			(hide yes)
 			(show_name no)
@@
 			)
 		)
-		(property "Datasheet" "https://www.lcsc.com/datasheet/lcsc_datasheet_2304140030_YAGEO-RC0402FR-0749K9L_C137969.pdf"
-			(at 38.1 207.01 0)
+		(property "Datasheet" "https://www.lcsc.com/datasheet/lcsc_datasheet_2411221126_UNI-ROYAL-Uniroyal-Elec-0402WGF1002TCE_C25744.pdf"
+			(at 38.1 204.47 0)
 			(hide yes)
 			(show_name no)
@@
 		)
 		(property "Description" "Resistor"
-			(at 38.1 207.01 0)
+			(at 38.1 204.47 0)
 			(hide yes)
 			(show_name no)
@@
 			)
 		)
-		(property "LCSC" "C137969"
-			(at 38.1 207.01 0)
+		(property "LCSC" "C25744"
+			(at 38.1 204.47 0)
 			(hide yes)
 			(show_name no)
@@
 			)
 		)
-		(property "MPN" "RC0402FR-0749K9L"
-			(at 38.1 207.01 0)
+		(property "MPN" "0402WGF1002TCE"
+			(at 38.1 204.47 0)
 			(hide yes)
 			(show_name no)
@@
 			)
 		)
-		(property "Manufacturer" "YAGEO"
-			(at 38.1 207.01 0)
+		(property "Manufacturer" "UNI-ROYAL(Uniroyal Elec)"
+			(at 38.1 204.47 0)
 			(hide yes)
 			(show_name no)
