File: hardware/iasis/iasis.kicad_sch (KiCad schematic)
At the start: 0 parts

Commit message: Add the CM5 carrier design for reference
The first board revision: a Raspberry Pi CM5 carrier with M.2 NVMe,
Ethernet and five USB 3 and USB-PD ports, as it stood before the compact
hub replaced it, squashed from 45 commits.
Other:
- sheet Host power and target budget renamed Logic power selection
- sheet Optional USB-C charging input renamed 24V input protection
- removed sheet Power control outputs
- added sheet 5V_AUX supply (power-5v-aux.kicad_sch)
- added sheet 5V_CM5 supply (power-5v-cm5.kicad_sch)
- added sheet CM5 carrier (carrier.kicad_sch)
- note added: "24 V input protection"
- note added: "24V_SYS"
- note added: "24V_SYS → 5V_AUX"
- note added: "24V_SYS → 5V_CM5"
- note added: "3V3_AON and hub supplies"
- note added: "5 V auxiliary"
- note added: "5 V compute supply"
- note added: "Adapter / host → 5V_LOGIC"
- note added: "Buttons and indicators"
- note added: "Compute Module 5"
- note added: "Control and monitoring"
- note added: "Dashed lines show functional relationships, not electrical nets."
- note added: "Ethernet, NVMe and recovery"
- note added: "External host / service USB"
- note added: "Five target ports"
- note added: "Functional overview; electrical connections on circuit sheets"
- note added: "I2C and isolation"
- note added: "Logic and hub rails"
- note added: "Logic source selection"
- note added: "One shared circuit × five"
- note added: "PD buses and GPIO expansion"
- note added: "PD policy and fault handling"
- note added: "Power distribution"
- note added: "Protected ADC inputs"
- note added: "RP2354 controller"
- note added: "Selected host to downstream"
- note added: "Temperature sensing"
- note added: "Two converter regions"
- note added: "USB data and host"
- note added: "USB host selection"
- note added: "USB hub and selection"
- note added: "Upstream USB-C"
- note added: "User controls and status"
- note added: "Voltage and current"
- note added: "iasis — system overview"
- note removed: "3.3 V, hub core rail and hardware reset"
- note removed: "Charging-stage temperature measurements"
- note removed: "Common hub and control circuitry with an optional five-port charging population"
- note removed: "Control and recovery"
- note removed: "External USB host: data, CC and 5 V presence"
- note removed: "Five identical USB-C / DFU / power channels"
- note removed: "Host / target status and deliberate confirmation"
- note removed: "Host-powered logic and bounded target supply"
- note removed: "IASIS — USB-C DFU hub"
- note removed: "Independent target VBUS measurements"
- note removed: "Monitoring"
- note removed: "Optional USB-C charging power input"
- note removed: "Per-port I2C, display and UART debug"
- note removed: "Power"
- note removed: "RP2354, USB recovery and SWD"
- note removed: "USB data"
- note removed: "USB7206C: five target ports and MCU USB2"
