File: hardware/iasis/iasis.kicad_sch (KiCad schematic)
At the start: 0 parts

Commit message: Wire the schematic islands and side-match the RP2354 GPIOs
Each sheet now draws its circuits with wires. Labels remain at block edges
and on single-part islands: buttons, test points, decoupling and pull
resistors. The target-port page wires its hierarchical labels straight to
the child sheet pins, the ports page points its labels away from each
block, and the root sheet keeps every block clear of the title block.

The RP2354B GPIOs are reassigned so each signal leaves the package on the
side facing its destination. Update PCB from Schematic applied the 43
U1101 pad-net changes with no geometry change. Otherwise the netlist
matches the previous design, ERC keeps its 14 existing warnings and DRC
reports no parity issues.
Other:
- note added: "Discharge, 9 V select and host budget outputs"
- note added: "Monitoring and power control"
- note removed: "Monitoring"
Changed lines of the file:
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@@
 	(text "Power"
 		(exclude_from_sim no)
-		(at 25 230 0)
+		(at 25 210 0)
 		(effects
 			(font
@@
 	(text "RP2354, USB recovery and SWD"
 		(exclude_from_sim no)
-		(at 30 170 0)
+		(at 30 160 0)
 		(effects
 			(font
@@
 	(text "Host / target status and deliberate confirmation"
 		(exclude_from_sim no)
-		(at 390 170 0)
+		(at 390 160 0)
 		(effects
 			(font
@@
 	(text "Independent target VBUS measurements"
 		(exclude_from_sim no)
-		(at 30 350 0)
+		(at 30 320 0)
 		(effects
 			(font
@@
 	(text "3.3 V, hub core rail and hardware reset"
 		(exclude_from_sim no)
-		(at 210 260 0)
+		(at 210 240 0)
 		(effects
 			(font
@@
 	(text "Per-port I2C, display and UART debug"
 		(exclude_from_sim no)
-		(at 210 170 0)
+		(at 210 160 0)
 		(effects
 			(font
@@
 	(text "Host-powered logic and bounded target supply"
 		(exclude_from_sim no)
-		(at 30 260 0)
+		(at 30 240 0)
 		(effects
 			(font
@@
 	(text "Control and recovery"
 		(exclude_from_sim no)
-		(at 25 140 0)
+		(at 25 130 0)
 		(effects
 			(font
@@
 	(text "Charging-stage temperature measurements"
 		(exclude_from_sim no)
-		(at 210 350 0)
-		(effects
-			(font
-				(size 1.8 1.8)
-			)
-			(justify left top)
-		)
-	)
-	(text "Monitoring"
-		(exclude_from_sim no)
-		(at 25 320 0)
+		(at 210 320 0)
+		(effects
+			(font
+				(size 1.8 1.8)
+			)
+			(justify left top)
+		)
+	)
+	(text "Monitoring and power control"
+		(exclude_from_sim no)
+		(at 25 290 0)
 		(effects
 			(font
@@
 	(text "Optional USB-C charging power input"
 		(exclude_from_sim no)
-		(at 390 260 0)
+		(at 390 240 0)
+		(effects
+			(font
+				(size 1.8 1.8)
+			)
+			(justify left top)
+		)
+	)
+	(text "Discharge, 9 V select and host budget outputs"
+		(exclude_from_sim no)
+		(at 390 320 0)
 		(effects
 			(font
@@
 	)
 	(sheet
-		(at 385 245)
+		(at 385 225)
 		(size 160 40)
 		(exclude_from_sim no)
@@
 		)
 		(property "Sheetname" "Optional USB-C charging input"
-			(at 385 242.46 0)
+			(at 385 224.2884 0)
 			(show_name no)
 			(do_not_autoplace no)
@@
 		)
 		(property "Sheetfile" "power-input.kicad_sch"
-			(at 385 287.54 0)
+			(at 385 265.5884 0)
 			(show_name no)
 			(do_not_autoplace no)
@@
 	)
 	(sheet
-		(at 25 155)
+		(at 25 145)
 		(size 160 40)
 		(exclude_from_sim no)
@@
 		)
 		(property "Sheetname" "RP2354 controller"
-			(at 25 152.46 0)
+			(at 25 144.2884 0)
 			(show_name no)
 			(do_not_autoplace no)
@@
 		)
 		(property "Sheetfile" "controller-core.kicad_sch"
-			(at 25 197.54 0)
+			(at 25 185.5884 0)
 			(show_name no)
 			(do_not_autoplace no)
@@
 	)
 	(sheet
-		(at 385 335)
-		(size 165 50)
+		(at 385 305)
+		(size 160 40)
 		(exclude_from_sim no)
 		(in_bom yes)
@@
 		)
 		(property "Sheetname" "Power control outputs"
-			(at 385 332.46 0)
+			(at 385 304.2884 0)
 			(show_name no)
 			(do_not_autoplace no)
@@
 		)
 		(property "Sheetfile" "controller-power.kicad_sch"
-			(at 385 387.54 0)
+			(at 385 345.5884 0)
 			(show_name no)
 			(do_not_autoplace no)
@@
 	)
 	(sheet
-		(at 205 335)
+		(at 205 305)
 		(size 160 40)
 		(exclude_from_sim no)
@@
 		)
 		(property "Sheetname" "Converter temperatures"
-			(at 205 332.46 0)
+			(at 205 304.2884 0)
 			(show_name no)
 			(do_not_autoplace no)
@@
 		)
 		(property "Sheetfile" "controller-temperature.kicad_sch"
-			(at 205 377.54 0)
+			(at 205 345.5884 0)
 			(show_name no)
 			(do_not_autoplace no)
@@
 	)
 	(sheet
-		(at 25 335)
+		(at 25 305)
 		(size 160 40)
 		(exclude_from_sim no)
@@
 		)
 		(property "Sheetname" "Port voltage measurement"
-			(at 25 332.46 0)
+			(at 25 304.2884 0)
 			(show_name no)
 			(do_not_autoplace no)
@@
 		)
 		(property "Sheetfile" "controller-sense.kicad_sch"
-			(at 25 377.54 0)
+			(at 25 345.5884 0)
 			(show_name no)
 			(do_not_autoplace no)
@@
 	)
 	(sheet
-		(at 205 245)
+		(at 205 225)
 		(size 160 40)
 		(exclude_from_sim no)
@@
 		)
 		(property "Sheetname" "Logic supplies and reset"
-			(at 205 242.46 0)
+			(at 205 224.2884 0)
 			(show_name no)
 			(do_not_autoplace no)
@@
 		)
 		(property "Sheetfile" "power-logic.kicad_sch"
-			(at 205 287.54 0)
+			(at 205 265.5884 0)
 			(show_name no)
 			(do_not_autoplace no)
@@
 	)
 	(sheet
-		(at 385 155)
+		(at 385 145)
 		(size 160 40)
 		(exclude_from_sim no)
@@
 		)
 		(property "Sheetname" "Indicators and confirmation"
-			(at 385 152.46 0)
+			(at 385 144.2884 0)
 			(show_name no)
 			(do_not_autoplace no)
@@
 		)
 		(property "Sheetfile" "controller-panel.kicad_sch"
-			(at 385 197.54 0)
+			(at 385 185.5884 0)
 			(show_name no)
 			(do_not_autoplace no)
@@
 		)
 		(property "Sheetname" "USB hub — ports 1–5"
-			(at 205 62.46 0)
+			(at 205 64.2884 0)
 			(show_name no)
 			(do_not_autoplace no)
@@
 		)
 		(property "Sheetfile" "hub.kicad_sch"
-			(at 205 107.54 0)
+			(at 205 105.5884 0)
 			(show_name no)
 			(do_not_autoplace no)
@@
 		)
 		(property "Sheetname" "Host port"
-			(at 25 62.46 0)
+			(at 25 64.2884 0)
 			(show_name no)
 			(do_not_autoplace no)
@@
 		)
 		(property "Sheetfile" "host-port.kicad_sch"
-			(at 25 107.54 0)
+			(at 25 105.5884 0)
 			(show_name no)
 			(do_not_autoplace no)
@@
 	)
 	(sheet
-		(at 25 245)
+		(at 25 225)
 		(size 160 40)
 		(exclude_from_sim no)
@@
 		)
 		(property "Sheetname" "Host power and target budget"
-			(at 25 242.46 0)
+			(at 25 224.2884 0)
 			(show_name no)
 			(do_not_autoplace no)
@@
 		)
 		(property "Sheetfile" "power-select.kicad_sch"
-			(at 25 287.54 0)
+			(at 25 265.5884 0)
 			(show_name no)
 			(do_not_autoplace no)
@@
 		)
 		(property "Sheetname" "Target ports"
-			(at 385 62.46 0)
+			(at 385 64.2884 0)
 			(show_name no)
 			(do_not_autoplace no)
@@
 		)
 		(property "Sheetfile" "ports.kicad_sch"
-			(at 385 107.54 0)
+			(at 385 105.5884 0)
 			(show_name no)
 			(do_not_autoplace no)
@@
 	)
 	(sheet
-		(at 205 155)
+		(at 205 145)
 		(size 160 40)
 		(exclude_from_sim no)
@@
 		)
 		(property "Sheetname" "Management buses"
-			(at 205 152.46 0)
+			(at 205 144.2884 0)
 			(show_name no)
 			(do_not_autoplace no)
@@
 		)
 		(property "Sheetfile" "controller-bus.kicad_sch"
-			(at 205 197.54 0)
-			(show_name no)
-			(do_not_autoplace no)
+			(at 205 185.5884 0)
+			(show_name no)
+			(do_not_autoplace no)

Commit message: Redraw the root and target port hierarchy sheets
The root sheet groups the twelve function blocks into four rows by
area, each block described inside its frame. Sheet pins are justified
and ordered by signal flow, with USB data and the bus on the left and
control and status on the right.

After a native schematic save the netlist is identical (651 components,
541 nets), ERC still reports only the 14 PWR_FLAG pin-to-pin warnings,
and Update PCB from Schematic previews no actions.
Other:
- title: (none) -> IASIS — USB-C DFU hub
