File: hardware/iasis/power-select.kicad_sch (KiCad schematic)
At the start: 23 parts, among them Q1911 2N7002, Q1912 2N7002, U1901 AP22653W6-7, U1902 TPS259470LRPWR

Commit message: Add the CM5 carrier design for reference
The first board revision: a Raspberry Pi CM5 carrier with M.2 NVMe,
Ethernet and five USB 3 and USB-PD ports, as it stood before the compact
hub replaced it, squashed from 45 commits.
Parts:
- removed C1911, C1913: 100n, Capacitor_SMD:C_0402_1005Metric, symbol Device:C
- removed C1912: 10u 16V X5R, Capacitor_SMD:C_0805_2012Metric, symbol Device:C
- removed Q1911, Q1912: 2N7002, Package_TO_SOT_SMD:SOT-23, symbol Transistor_FET:2N7002
- removed R1911, R1915, R1917: 100k, Resistor_SMD:R_0402_1005Metric, symbol Device:R
- removed R1912: 10k, Resistor_SMD:R_0402_1005Metric, symbol Device:R
- removed R1913: 200k 1%, Resistor_SMD:R_0402_1005Metric, symbol Device:R
- removed R1914: 68k 1%, Resistor_SMD:R_0402_1005Metric, symbol Device:R
- removed R1916: 22k 1%, Resistor_SMD:R_0402_1005Metric, symbol Device:R
- removed U1901: AP22653W6-7, Package_TO_SOT_SMD:SOT-23-6, symbol Iasis:AP22653W6-7
- added C1901: 1n 50V C0G, Capacitor_SMD:C_0402_1005Metric, symbol Device:C
- added C1902: 100n, Capacitor_SMD:C_0402_1005Metric, symbol Device:C
- added D1902: SS34, Diode_SMD:D_SMA, symbol Diode:SS34
- added Q1901: 2N7002, Package_TO_SOT_SMD:SOT-23, symbol Transistor_FET:2N7002
- added R1901: 68k 1%, Resistor_SMD:R_0402_1005Metric, symbol Device:R
- added R1902: 6.8k 1%, Resistor_SMD:R_0402_1005Metric, symbol Device:R
- added R1903: 20k 1%, Resistor_SMD:R_0402_1005Metric, symbol Device:R
- added R1904: 4.7k, Resistor_SMD:R_0402_1005Metric, symbol Device:R
- added R1905: 1.5k 1%, Resistor_SMD:R_0402_1005Metric, symbol Device:R
- added U1901: TPS259470LRPWR, Iasis:TI_RPW0010A, symbol Iasis:TPS259470LRPWR
- C1903: LCSC C1622 -> (none); MPN CL10B473KB8NNNC -> (none); Manufacturer Samsung Electro-Mechanics -> (none); Population Common -> (none)
- C1904: Manufacturer Samsung Electro-Mechanics -> (none); Population Common -> (none)
- C1905: LCSC C55530 -> (none); MPN CL32B226KOJNNNE -> (none); Manufacturer Samsung Electro-Mechanics -> (none); Population Common -> (none)
- C1906: LCSC C1525 -> (none); MPN CL05B104KO5NNNC -> (none); Manufacturer Samsung Electro-Mechanics -> (none); Population Common -> (none)
- R1906: LCSC C36871 -> (none); MPN 0402WGF6802TCE -> (none); Manufacturer UNI-ROYAL(Uniroyal Elec) -> (none); Population Common -> (none)
- R1907: LCSC C25744 -> (none); MPN 0402WGF1002TCE -> (none); Manufacturer UNI-ROYAL(Uniroyal Elec) -> (none); Population Common -> (none)
- R1908: LCSC C25765 -> (none); MPN 0402WGF2002TCE -> (none); Manufacturer UNI-ROYAL(Uniroyal Elec) -> (none); Population Common -> (none)
- R1909: LCSC C11702 -> (none); MPN 0402WGF1001TCE -> (none); Manufacturer UNI-ROYAL(Uniroyal Elec) -> (none); Population Common -> (none)
- R1910: LCSC C25076 -> (none); MPN 0402WGF1000TCE -> (none); Manufacturer UNI-ROYAL(Uniroyal Elec) -> (none); Population Common -> (none)
- U1902: LCSC C3662793 -> (none); MPN TPS259470LRPWR -> (none); Manufacturer Texas Instruments -> (none); Population Common -> (none)
Connections:
- net 5V_LOGIC: now also D1902.2 (A), U1901.6 (OUT)
- net EXT_VBUS: now also Q1901.3 (D)
- net GND: now also C1901.2, C1902.2, R1903.2, R1905.2, U1901.8 (GND)
- net AUX_DVDT_C: now reaches C1903.1, R1910.2
- net LOGIC_DVDT renamed AUX_DVDT
- net LOGIC_EN renamed AUX_EN
- net LOGIC_ILIM renamed AUX_ILM
- net LOGIC_OVLO renamed AUX_OVLO
- net AUX_OVLO: now also Q1901.2 (S)
- new net 24V_SYS: D1902.1 (K)
- new net 5V_AUX: C1902.1, R1901.1, R1904.1, U1901.5 (IN)
- new net PRI_AUXOFF: Q1901.1 (G), R1904.2, U1901.3 (AUXOFF)
- new net PRI_DVDT: C1901.1, U1901.7 (DVDT)
- new net PRI_EN: R1901.2, R1902.1, U1901.1 (EN_UVLO)
- new net PRI_ILM: R1905.1, U1901.9 (ILM)
- new net PRI_OVLO: R1902.2, R1903.1, U1901.2 (OVLO)
- no-connect marks 3 -> 5
Other:
- note added: "5V_LOGIC — adapter or host power for the logic"
- note added: "Adapter (primary)"
- note added: "Host VBUS (auxiliary)"
- note added: "Priority mux per TI SLVSFC9C 8.2.5, option 2: while 5V_AUX is valid, AUXOFF turns Q1901 on and EXT_VBUS holds the auxiliary OVLO high. Without a host nothing drives EXT_VBUS: AUXOFF only reaches Q1901's gate, and Q1901 then ties EXT_VBUS to R1908. Primary: UVLO 4.24V rising, OVLO 5.69V, ILM 2.2A. Auxiliary: UVLO 3.92V rising, OVLO 5.88V, ILM 3.3A. Auxiliary dVdt 0.043V/ms keeps bus-powered inrush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"
- note removed: "68k / 22k selections: 00 ≤0.17 A; 10 ≤0.55 A; 01 ≤1.45 A; 11 ≤1.89 A. Budget the worst tier plus logic consumption. No automatic 3 A assumption. Target aggregate defaults off; the hub and MCU remain powered upstream of it."
- note removed: "Host power — autonomous logic and bounded target allocation"
- note removed: "Logic starts from host VBUS. The MCU enables target power only after the upstream current allowance is known."
- moved on the sheet: C1903, C1904, C1905, C1906, R1906, R1907, R1908, R1909, R1910, U1902
