File: hardware/iasis/target-power.kicad_sch (KiCad schematic)
At the start: 18 parts, among them Q1221 2N7002, U1202 TPS259470LRPWR, U1203 SN74LVC2G08DCUR

Commit message: Add the CM5 carrier design for reference
The first board revision: a Raspberry Pi CM5 carrier with M.2 NVMe,
Ethernet and five USB 3 and USB-PD ports, as it stood before the compact
hub replaced it, squashed from 45 commits.
Parts:
- removed Q1221: 2N7002, Package_TO_SOT_SMD:SOT-23, symbol Transistor_FET:2N7002
- removed R1221, R1223: 100k, Resistor_SMD:R_0402_1005Metric, symbol Device:R
- removed R1222: 1k 1%, Resistor_SMD:R_0805_2012Metric, symbol Device:R
- removed U1203: SN74LVC2G08DCUR, Package_SO:VSSOP-8_2.3x2mm_P0.5mm, symbol 74xGxx:74LVC2G08
- added C1201: 4.7n, Capacitor_SMD:C_0402_1005Metric, symbol Device:C
- added C1202: 100p C0G, Capacitor_SMD:C_0402_1005Metric, symbol Device:C
- added C1203, C1204: 100n 16V X7R, Capacitor_SMD:C_0603_1608Metric, symbol Device:C
- added C1205: 22u 16V X7R, Capacitor_SMD:C_1210_3225Metric, symbol Device:C
- added C1206: 100n, Capacitor_SMD:C_0402_1005Metric, symbol Device:C
- added C1207, C1208, C1211, C1212, C1213, C1214: 10u 50V X7R, Capacitor_SMD:C_1210_3225Metric, symbol Device:C
- added C1209: 100n 50V X7R, Capacitor_SMD:C_0603_1608Metric, symbol Device:C
- added C1210: 100u 50V, Capacitor_SMD:CP_Elec_10x10.5, symbol Device:C_Polarized
- added C1215: 220u 25V, Capacitor_SMD:CP_Elec_8x10.5, symbol Device:C_Polarized
- added L1201: SRP1265A-4R7M, Iasis:Bourns_SRP1265A, symbol Device:L
- added Q1201, Q1202: CSD18543Q3A, Iasis:TI_CSD18543Q3A, symbol Transistor_FET:CSD18543Q3A
- added R1201, R1202: 0, Resistor_SMD:R_0402_1005Metric, symbol Device:R
- added R1203: 10m 1% 1W, Iasis:Yageo_PA1206_4-20mOhm, symbol Device:R
- added R1204: 100k, Resistor_SMD:R_0402_1005Metric, symbol Device:R
- added R1205: 49.9k 1%, Resistor_SMD:R_0402_1005Metric, symbol Device:R
- added R1206: 1 1%, Resistor_SMD:R_0402_1005Metric, symbol Device:R
- added R1207: 60.4k 1%, Resistor_SMD:R_0402_1005Metric, symbol Device:R
- added R1208: 56.2k 1%, Resistor_SMD:R_0402_1005Metric, symbol Device:R
- added U1201: TPS55288RPMR, Iasis:TI_RPM0026A, symbol Iasis:TPS55288RPMR
- added U1203: SN74AUP1G08DBVR, Package_TO_SOT_SMD:SOT-23-5, symbol 74xGxx:74AUP1G08
- C1216: LCSC C1525 -> (none); MPN CL05B104KO5NNNC -> (none); Manufacturer Samsung Electro-Mechanics -> (none); Population Common -> (none)
- C1217: LCSC C525198 -> (none); MPN FN15N102J500PNG -> (none); Manufacturer PSA(Prosperity Dielectrics) -> (none); Population Common -> (none)
- C1218: value 2.2u 25V X5R -> 10u 50V X7R; footprint Capacitor_SMD:C_0603_1608Metric -> Capacitor_SMD:C_1210_3225Metric; LCSC C57895 -> (none); MPN CL10A225KA8NNNC -> (none); Manufacturer Samsung Electro-Mechanics -> (none); Population Common -> (none)
- C1219, C1220: footprint Capacitor_SMD:C_0402_1005Metric -> Capacitor_SMD:C_0603_1608Metric; LCSC C307331 -> (none); MPN CL05B104KB54PNC -> (none); Manufacturer Samsung Electro-Mechanics -> (none); Population Common -> (none)
- R1209, R1215: LCSC C25741 -> (none); MPN 0402WGF1003TCE -> (none); Manufacturer UNI-ROYAL(Uniroyal Elec) -> (none); Population Common -> (none)
- R1210, R1212: LCSC C25744 -> (none); MPN 0402WGF1002TCE -> (none); Manufacturer UNI-ROYAL(Uniroyal Elec) -> (none); Population Common -> (none)
- R1211: value 39k 1% -> 174k 1%; LCSC C25783 -> (none); MPN 0402WGF3902TCE -> (none); Manufacturer UNI-ROYAL(Uniroyal Elec) -> (none); Population Common -> (none)
- R1213: value 6.49k 1% -> 806 1%; LCSC C364360 -> C11522; MPN RC0402FR-076K49L -> RTT028060FTH; Manufacturer YAGEO -> (none); Population Common -> (none)
- R1214: value 100k -> 1k 1% 1W; footprint Resistor_SMD:R_0402_1005Metric -> Resistor_SMD:R_2512_6332Metric; LCSC C25741 -> C3017416; MPN 0402WGF1003TCE -> SCR2512F1K; Manufacturer UNI-ROYAL(Uniroyal Elec) -> VO; Population Common -> (none)
- U1202: LCSC C3662793 -> (none); MPN TPS259470LRPWR -> (none); Manufacturer Texas Instruments -> (none); Population Common -> (none)
Connections:
- net 3V3_AON: now also U1203.5 (VCC)
- net CC_FAULT_N: now also U1203.2
- net GND: now also C1201.2, C1202.2, C1205.2, C1206.2, C1207.2, C1208.2, C1209.2, C1210.2, C1211.2, C1212.2, C1213.2, C1214.2, C1215.2, Q1202.1 (S), Q1202.2 (S), Q1202.3 (S), R1204.2, R1205.2, R1207.2, U1201.10 (AGND), U1201.24 (PGND), U1201.7 (DITH_SYNC), U1201.9 (PGND), U1203.3 (GND)
- net POWER_FAULT_N: now also U1201.14 (FB_INT)
- net HOST_DVDT renamed DVDT
- net HOST_EN renamed OUTPUT_EN
- net OUTPUT_EN: now also U1203.4
- net HOST_EN_REQ renamed OUTPUT_EN_REQ
- net OUTPUT_EN_REQ: now also U1203.1
- net HOST_ILIM renamed ILM
- net HOST_OVLO renamed OVLO
- net HOST_TARGET_5V renamed EFUSE_IN
- net EFUSE_IN: now also R1203.2, U1201.13 (ISN)
- new net 24V_SYS: C1207.1, C1208.1, C1209.1, C1210.1, Q1201.5 (D), U1201.3 (VIN)
- new net 5V_LOGIC: R1206.2
- new net BOOT1: C1203.1, U1201.22 (BOOT1)
- new net BOOT2: C1204.1, U1201.20 (BOOT2)
- new net COMP: C1202.1, R1208.1, U1201.18 (COMP)
- new net COMP_RC: C1201.1, R1208.2
- new net CONVERTER_EN: R1204.1, U1201.4 (EN_UVLO)
- new net DR1H: R1201.1, U1201.2 (DR1H)
- new net DR1L: R1202.1, U1201.1 (DR1L)
- new net FSW: R1205.1, U1201.8 (FSW)
- new net GATE_H: Q1201.4 (G), R1201.2
- new net GATE_L: Q1202.4 (G), R1202.2
- new net ILIM: R1207.1, U1201.17 (ILIM)
- new net SCL: U1201.5 (SCL)
- new net SDA: U1201.6 (SDA)
- new net SW1: C1203.2, L1201.1, Q1201.1 (S), Q1201.2 (S), Q1201.3 (S), Q1202.5 (D), U1201.23 (SW1)
- new net SW2: C1204.2, L1201.2, U1201.21 (SW2), U1201.25 (SW2)
- new net VCC: C1205.1, C1206.1, R1206.1, U1201.19 (VCC)
- new net VOUT: C1211.1, C1212.1, C1213.1, C1214.1, C1215.1, R1203.1, U1201.11 (VOUT), U1201.12 (ISP), U1201.26 (VOUT)
- no-connect marks 2 -> 4
Other:
- removed sheet Optional charging
- note added: "24V input bypass"
- note added: "Before output enable: EN high, OE=0, DISCHG=1 for at least 200ms; program 5.1V, OE=1, settle, then enable the eFuse. Verify connector VBUS before attachment / PD progression. Both enables default low. Firmware latches faults and removes both enables."
- note added: "Converter compensation"
- note added: "Converter output bypass"
- note added: "Current sense and protected output"
- note added: "External half bridge"
- note added: "Hardware output interlock"
- note added: "Kelvin-route current-sense leads from the inner shunt lands. Keep switching loops short."
- note added: "MODE open: VCC from 5V_LOGIC through the 1 ohm feed; I2C address 0x75; PFM."
- note added: "Programmable buck-boost converter"
- note added: "Protected VBUS and discharge"
- note added: "VCC from 5V_LOGIC"
- note removed: "HOST_TARGET_5V feeds a reverse-blocking switch; optional charging joins only at VBUS."
- note removed: "Host branch: ~0.5 A per-port limit; the common limiter owns the total host budget. Both branches must be off before active discharge. CC protection gates both source enables in hardware. 100k remains across VBUS when all active circuitry is off."
- note removed: "Hub: entire child DNP. HubPD: converter and protected source fitted."
- note removed: "Target output — common host branch, gating and discharge"
- title: (none) -> Programmable port supply
- moved on the sheet: C1216, C1217, C1218, C1219, C1220, R1209, R1210, R1211, R1212, R1213, R1214, R1215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
