File: hardware/iasis/target-power.kicad_sch (KiCad schematic)
At the start: 18 parts, among them Q1221 2N7002, U1202 TPS259470LRPWR, U1203 SN74LVC2G08DCUR

Commit message: Wire the schematic islands and side-match the RP2354 GPIOs
Each sheet now draws its circuits with wires. Labels remain at block edges
and on single-part islands: buttons, test points, decoupling and pull
resistors. The target-port page wires its hierarchical labels straight to
the child sheet pins, the ports page points its labels away from each
block, and the root sheet keeps every block clear of the title block.

The RP2354B GPIOs are reassigned so each signal leaves the package on the
side facing its destination. Update PCB from Schematic applied the 43
U1101 pad-net changes with no geometry change. Otherwise the netlist
matches the previous design, ERC keeps its 14 existing warnings and DRC
reports no parity issues.
Other:
- moved on the sheet: C1216, C1217, C1218, C1219, C1220, Q1221, R1209, R1210, R1211, R1212, R1213, R1214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

Commit message: Redraw the target port sheets
The per-port data, output and charging sheets follow the signal and
power paths left to right. The receptacle sits at the right edge with
its CC and USB 2 protection wired to it, the SuperSpeed mux and ESD
arrays below, and the charging buck, feedback divider, OVP network and
output eFuse in one row. The port sheet joins its two blocks with
wires. The netlist is unchanged.
Other:
- title: (none) -> Target output — common host branch, gating and discharge
- moved on the sheet: C1216, C1217, C1218, C1219, C1220, Q1221, R1209, R1210, R1211, R1212, R1213, R1214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

Commit message: Fit Nexperia 74LVC2G08DC-Q100H as the target-port AND gates
JLC stock of SN74LVC2G08DCUR (C91875) fell to 20, short of the 25 a
five-board order places. Nexperia's 74LVC2G08DC-Q100H (C548572, 2,920
in stock, $0.18 against $0.39) has the same pinout, IOFF and supply
range, in SOT765-1. That and TI's DCU are both JEDEC MO-187, so the
footprint, placement and copper stay as they are.

U1203, U1303, U1403, U1503 and U1603 change Value, LCSC, MPN,
Manufacturer, Datasheet and Description only; the old Description
still named a single gate.

Netlist connectivity identical (651 components, 541 nets). ERC 14 as
before. DRC with refill and parity: 0 errors, 0 warnings,
0 unconnected.
Parts:
- U1203: value SN74LVC2G08DCUR -> 74LVC2G08DC-Q100H; LCSC C91875 -> C548572; MPN SN74LVC2G08DCUR -> 74LVC2G08DC-Q100H; Manufacturer Texas Instruments -> Nexperia
Changed lines of the file:
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@@
 			)
 		)
-		(property "Value" "SN74LVC2G08DCUR"
+		(property "Value" "74LVC2G08DC-Q100H"
 			(at 66.04 93.98 0)
 			(show_name no)
@@
 			)
 		)
-		(property "Datasheet" "https://www.ti.com/lit/ds/symlink/sn74lvc2g08.pdf"
+		(property "Datasheet" "https://assets.nexperia.com/documents/data-sheet/74LVC2G08_Q100.pdf"
 			(at 73.66 91.44 0)
 			(hide yes)
@@
 			)
 		)
-		(property "Description" "Single 2-input AND gate, low-power CMOS"
+		(property "Description" "Dual AND Gate, Low-Voltage CMOS"
 			(at 73.66 91.44 0)
 			(hide yes)
@@
 			)
 		)
-		(property "LCSC" "C91875"
+		(property "LCSC" "C548572"
 			(at 73.66 91.44 0)
 			(hide yes)
@@
 			)
 		)
-		(property "MPN" "SN74LVC2G08DCUR"
+		(property "MPN" "74LVC2G08DC-Q100H"
 			(at 73.66 91.44 0)
 			(hide yes)
@@
 			)
 		)
-		(property "Manufacturer" "Texas Instruments"
+		(property "Manufacturer" "Nexperia"
 			(at 73.66 101.6 0)
 			(hide yes)
@@
 			)
 		)
-		(property "Value" "SN74LVC2G08DCUR"
+		(property "Value" "74LVC2G08DC-Q100H"
 			(at 66.04 68.58 0)
 			(show_name no)
@@
 			)
 		)
-		(property "Datasheet" "https://www.ti.com/lit/ds/symlink/sn74lvc2g08.pdf"
+		(property "Datasheet" "https://assets.nexperia.com/documents/data-sheet/74LVC2G08_Q100.pdf"
 			(at 73.66 66.04 0)
 			(hide yes)
@@
 			)
 		)
-		(property "Description" "Single 2-input AND gate, low-power CMOS"
+		(property "Description" "Dual AND Gate, Low-Voltage CMOS"
 			(at 73.66 66.04 0)
 			(hide yes)
@@
 			)
 		)
-		(property "LCSC" "C91875"
+		(property "LCSC" "C548572"
 			(at 73.66 66.04 0)
 			(hide yes)
@@
 			)
 		)
-		(property "MPN" "SN74LVC2G08DCUR"
+		(property "MPN" "74LVC2G08DC-Q100H"
 			(at 73.66 66.04 0)
 			(hide yes)
@@
 			)
 		)
-		(property "Manufacturer" "Texas Instruments"
+		(property "Manufacturer" "Nexperia"
 			(at 73.66 76.2 0)
 			(hide yes)
@@
 			)
 		)
-		(property "Value" "SN74LVC2G08DCUR"
+		(property "Value" "74LVC2G08DC-Q100H"
 			(at 67.31 130.81 0)
 			(show_name no)
@@
 			)
 		)
-		(property "Datasheet" "https://www.ti.com/lit/ds/symlink/sn74lvc2g08.pdf"
+		(property "Datasheet" "https://assets.nexperia.com/documents/data-sheet/74LVC2G08_Q100.pdf"
 			(at 73.66 119.38 0)
 			(hide yes)
@@
 			)
 		)
-		(property "Description" "Single 2-input AND gate, low-power CMOS"
+		(property "Description" "Dual AND Gate, Low-Voltage CMOS"
 			(at 73.66 119.38 0)
 			(hide yes)
@@
 			)
 		)
-		(property "LCSC" "C91875"
+		(property "LCSC" "C548572"
 			(at 73.66 119.38 0)
 			(hide yes)
@@
 			)
 		)
-		(property "MPN" "SN74LVC2G08DCUR"
+		(property "MPN" "74LVC2G08DC-Q100H"
 			(at 73.66 119.38 0)
 			(hide yes)
@@
 			)
 		)
-		(property "Manufacturer" "Texas Instruments"
+		(property "Manufacturer" "Nexperia"
 			(at 73.66 129.54 0)
 			(hide yes)
