File: hardware/iasis/ports.kicad_sch (KiCad schematic)
At the start: 0 parts

Commit message: Redraw the root and target port hierarchy sheets
The root sheet groups the twelve function blocks into four rows by
area, each block described inside its frame. Sheet pins are justified
and ordered by signal flow, with USB data and the bus on the left and
control and status on the right.

After a native schematic save the netlist is identical (651 components,
541 nets), ERC still reports only the 14 PWR_FLAG pin-to-pin warnings,
and Update PCB from Schematic previews no actions.
Other:
- title: (none) -> Five independent target channels
