File: hardware/iasis/target-charge.kicad_sch (KiCad schematic)
At the start: 37 parts, among them Q1230 2N7002, Q1231 2N7002, Q1232 2N7002, U1230 LMR51450SDRRR, U1231 TPS26600PWPR, U1232 LM4040DIM3X-2.5/NOPB

Commit message: Wire the schematic islands and side-match the RP2354 GPIOs
Each sheet now draws its circuits with wires. Labels remain at block edges
and on single-part islands: buttons, test points, decoupling and pull
resistors. The target-port page wires its hierarchical labels straight to
the child sheet pins, the ports page points its labels away from each
block, and the root sheet keeps every block clear of the title block.

The RP2354B GPIOs are reassigned so each signal leaves the package on the
side facing its destination. Update PCB from Schematic applied the 43
U1101 pad-net changes with no geometry change. Otherwise the netlist
matches the previous design, ERC keeps its 14 existing warnings and DRC
reports no parity issues.
Connections:
- no-connect marks 4 -> 2
Other:
- moved on the sheet: C1230, C1231, C1232, C1233, C1234, C1235, C1236, C1237, C1238, C1239, L1230, Q1230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

Commit message: Redraw the target port sheets
The per-port data, output and charging sheets follow the signal and
power paths left to right. The receptacle sits at the right edge with
its CC and USB 2 protection wired to it, the SuperSpeed mux and ESD
arrays below, and the charging buck, feedback divider, OVP network and
output eFuse in one row. The port sheet joins its two blocks with
wires. The netlist is unchanged.
Other:
- title: (none) -> Optional target charging — 5 V / 9 V
- moved on the sheet: C1230, C1231, C1232, C1233, C1234, C1235, C1236, C1237, C1238, C1239, L1230, Q1230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

Commit message: Drill every via and thermal via at 0.3 mm
JLC prices 0.2 and 0.25 mm holes as a small-via tier that also forces
TG155 and a 4-wire Kelvin test: $39.18 on a five-board order. With
every plated hole at 0.3 mm or more the board quotes in the standard
tier.

- 2,005 vias keep their pads (0.45, 0.55, 0.6 mm) and drill 0.3 mm.
- U201's VQFN-100, the WQFN-20 and the HTSSOP-16 ThermalVias
  footprints move to Iasis.pretty copies with 0.3 mm thermal vias
  (121 holes); the schematic links follow.
- Rules match JLC's published via limits: 0.2 mm via hole to copper
  and hole to hole, 0.075 mm annular ring, 0.3 mm minimum hole.

DRC with refill and parity: 0 errors, 0 warnings, 0 unconnected.
Pour island counts unchanged; ERC unchanged at 14.
Parts:
- U1231: footprint Package_SO:HTSSOP-16-1EP_4.4x5mm_P0.65mm_EP3.4x5mm_Mask2.66x2.46mm_ThermalVias -> Iasis:HTSSOP-16-1EP_4.4x5mm_P0.65mm_EP3.4x5mm_Mask2.66x2.46mm_ThermalVias
Changed lines of the file:
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@@
 			)
 		)
-		(property "Footprint" "Package_SO:HTSSOP-16-1EP_4.4x5mm_P0.65mm_EP3.4x5mm_Mask2.66x2.46mm_ThermalVias"
+		(property "Footprint" "Iasis:HTSSOP-16-1EP_4.4x5mm_P0.65mm_EP3.4x5mm_Mask2.66x2.46mm_ThermalVias"
 			(at 358.14 77.47 0)
 			(hide yes)

Commit message: Use smaller charge inductors and bulk capacitors, and solder pads for debug
The 6.8 uH PSTMAA666460 (12.5 A saturation) replaces the 10 uH 11 x 10 mm
inductor, a 6.3 mm 35 V hybrid capacitor the 10 mm 50 V bulk capacitor on
each charging buck, and an 8 mm 68 uF part the 100 uF on the charging input.
SWD and UART become three solder pads each in Raspberry Pi debug order.
Parts:
- C1234: value 100u 50V -> 100u 35V; footprint Capacitor_SMD:CP_Elec_10x10.5 -> Capacitor_SMD:CP_Elec_6.3x7.7; LCSC C109086 -> C454360; MPN EEHZA1H101P -> EEHZK1V101XP
- L1230: value 10u 10A -> 6.8u 12.5A; footprint Iasis:PSPMAA1040 -> Iasis:PSTMAA666460; LCSC C2983105 -> C55172548; MPN PSPMAA1040-100M-ANP -> PSTMAA666460-6R8MB
Changed lines of the file:
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@@
 			)
 		)
-		(property "Value" "10u 10A"
+		(property "Value" "6.8u 12.5A"
 			(at 151.13 82.55 90)
 			(show_name no)
@@
 			)
 		)
-		(property "Footprint" "Iasis:PSPMAA1040"
+		(property "Footprint" "Iasis:PSTMAA666460"
 			(at 153.67 85.09 0)
 			(hide yes)
@@
 			)
 		)
-		(property "Datasheet" "https://wmsc.lcsc.com/wmsc/upload/file/pdf/v2/lcsc/2207051830_PROD-Tech-PSPMAA1040-100M-ANP_C2983105.pdf"
+		(property "Datasheet" "https://datasheet.lcsc.com/datasheet/pdf/eae0dbe4b558713dce5995c355b822c6.pdf"
 			(at 153.67 85.09 0)
 			(hide yes)
@@
 			)
 		)
-		(property "LCSC" "C2983105"
+		(property "LCSC" "C55172548"
 			(at 153.67 85.09 0)
 			(hide yes)
@@
 			)
 		)
-		(property "MPN" "PSPMAA1040-100M-ANP"
+		(property "MPN" "PSTMAA666460-6R8MB"
 			(at 153.67 85.09 0)
 			(hide yes)
@@
 			)
 		)
-		(property "Value" "100u 50V"
+		(property "Value" "100u 35V"
 			(at 273.05 88.9 0)
 			(show_name no)
@@
 			)
 		)
-		(property "Footprint" "Capacitor_SMD:CP_Elec_10x10.5"
+		(property "Footprint" "Capacitor_SMD:CP_Elec_6.3x7.7"
 			(at 271.78 88.9 0)
 			(hide yes)
@@
 			)
 		)
-		(property "Datasheet" "https://www.lcsc.com/datasheet/lcsc_datasheet_2304140030_PANASONIC-EEHZA1H101P_C109086.pdf"
+		(property "Datasheet" "https://datasheet.lcsc.com/datasheet/pdf/8c74a3ab0c5c583fd1c39d99a73b3ca6.pdf"
 			(at 271.78 88.9 0)
 			(hide yes)
@@
 			)
 		)
-		(property "LCSC" "C109086"
+		(property "LCSC" "C454360"
 			(at 271.78 88.9 0)
 			(hide yes)
@@
 			)
 		)
-		(property "MPN" "EEHZA1H101P"
+		(property "MPN" "EEHZK1V101XP"
 			(at 271.78 88.9 0)
 			(hide yes)

Commit message: fix: use Economic-compatible Lelon bulk capacitors
Parts:
- C1234: LCSC C454360 -> C3031628; MPN EEHZK1V101XP -> HBO101M1VTR-0608; Manufacturer PANASONIC -> Lelon
Changed lines of the file:
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@@
 			)
 		)
-		(property "Datasheet" "https://datasheet.lcsc.com/datasheet/pdf/8c74a3ab0c5c583fd1c39d99a73b3ca6.pdf"
+		(property "Datasheet" "https://www.lelon.com.tw/upload/guides/2025%20%E7%94%B5%E5%AE%B9%E5%99%A8%E7%9B%AE%E5%BD%9520250123075950.pdf"
 			(at 271.78 88.9 0)
 			(hide yes)
@@
 			)
 		)
-		(property "LCSC" "C454360"
+		(property "LCSC" "C3031628"
 			(at 271.78 88.9 0)
 			(hide yes)
@@
 			)
 		)
-		(property "MPN" "EEHZK1V101XP"
+		(property "MPN" "HBO101M1VTR-0608"
 			(at 271.78 88.9 0)
 			(hide yes)
@@
 			)
 		)
-		(property "Manufacturer" "PANASONIC"
+		(property "Manufacturer" "Lelon"
 			(at 269.24 88.9 0)
 			(hide yes)
