File: hardware/lite/pcb/hub.kicad_sch (KiCad schematic)
At the start: 57 parts, among them U201 USB7206CT/KDX, U204 SN74AUP1G08DCKR, Y201 X322525MSB4SI

Commit message: feat(hardware): share brick power across ports and add CM5 link
A connected PD supply now runs the logic through its own buck and feeds
one TPS55288 buck-boost stage per port, so the contract is shared as
5-20 V at up to 5 A per port. The hub's VBUS detect becomes an OR gate,
a host-select mux lets a CM5 side board drive the hub over a 24-pin ZIF
link, and a CM5 variant joins Hub and HubPD.

The board is synced to the schematic and its old routing removed; the
new parts wait below the outline for placement.
Parts:
- removed R216: 10k, Resistor_SMD:R_0402_1005Metric, symbol Device:R
- added C224: 100n, Capacitor_SMD:C_0402_1005Metric, symbol Device:C
- added R231: 100k, Resistor_SMD:R_0402_1005Metric, symbol Device:R
- added R232: 200k 1%, Resistor_SMD:R_0402_1005Metric, symbol Device:R
- added U205: SN74LVC1G32DBVR, Package_TO_SOT_SMD:SOT-23-5, symbol 74xGxx:74LVC1G32
Connections:
- net 3V3_AON: now also C224.1, U205.5 (VCC)
- net GND: now also C224.2, R232.2, U205.3 (GND)
- net HUB_UP_VBUS: now also U205.4
- net EXT_D_N renamed HUB_D_N
- net EXT_D_P renamed HUB_D_P
- net EXT_RX_N renamed HUB_RX_N
- net EXT_RX_P renamed HUB_RX_P
- net EXT_TX_N renamed HUB_TX_N
- net EXT_TX_P renamed HUB_TX_P
- new net: R231.2, R232.1, U205.1
- new net CM5_HOST: U205.2
- new net EXT_VBUS: R231.1
Other:
- note added: "Configuration 3: CFG_STRAP1 10k; CFG_STRAP2/3, NON_REM and BC_EN 200k pull-downs. Internal ROM boot; all ports removable; battery charging detection off. HUB_SCL/SDA stay low during reset for autonomous attachment. RESET_N = AON_RESET_N AND HUB_RUN; HUB_RUN has a pull-up. The selected host reaches the hub through the host-select mux (host-port sheet). HUB_UP_VBUS = EXT_VBUS (divided) OR CM5_HOST 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"
- note removed: "Configuration 3: CFG_STRAP1 10k; CFG_STRAP2/3, NON_REM and BC_EN 200k pull-downs. Internal ROM boot; all ports removable; battery charging detection off. HUB_SCL/SDA stay low during reset for autonomous attachment. RESET_N = AON_RESET_N AND HUB_RUN; HUB_RUN has a pull-up. The external host reaches the hub directly through the upstream orientation mux. HUB_UP_VBUS has a 10k pull-up to 3V3_AON and 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"
- moved on the sheet: R217, R218, R219, R220, R221, R222, R223, R224, R225, R226, R227, R228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
