File: hardware/lite/pcb/ports.kicad_sch (KiCad schematic)
At the start: 0 parts

Commit message: feat(hardware): share brick power across ports and add CM5 link
A connected PD supply now runs the logic through its own buck and feeds
one TPS55288 buck-boost stage per port, so the contract is shared as
5-20 V at up to 5 A per port. The hub's VBUS detect becomes an OR gate,
a host-select mux lets a CM5 side board drive the hub over a 24-pin ZIF
link, and a CM5 variant joins Hub and HubPD.

The board is synced to the schematic and its old routing removed; the
new parts wait below the outline for placement.
Other:
- sheet Target 1 ports: added OV_HIGH; removed SEL_9V
- sheet Target 2 ports: added OV_HIGH; removed SEL_9V
- sheet Target 3 ports: added OV_HIGH; removed SEL_9V
- sheet Target 4 ports: added OV_HIGH; removed SEL_9V
- sheet Target 5 ports: added OV_HIGH; removed SEL_9V
