File: hardware/lite/pcb/target-power.kicad_sch (KiCad schematic)
At the start: 18 parts, among them Q1221 2N7002, U1202 TPS259470LRPWR, U1203 74LVC2G08DC-Q100H

Commit message: feat(hardware): share brick power across ports and add CM5 link
A connected PD supply now runs the logic through its own buck and feeds
one TPS55288 buck-boost stage per port, so the contract is shared as
5-20 V at up to 5 A per port. The hub's VBUS detect becomes an OR gate,
a host-select mux lets a CM5 side board drive the hub over a 24-pin ZIF
link, and a CM5 variant joins Hub and HubPD.

The board is synced to the schematic and its old routing removed; the
new parts wait below the outline for placement.
Parts:
- U1202: value TPS259470LRPWR -> TPS259470ARPWR; LCSC C3662793 -> C3662799; MPN TPS259470LRPWR -> TPS259470ARPWR
Other:
- sheet Optional charging ports: added OV_HIGH, POWER_FAULT_N, SCL, SDA; removed DISCHARGE, SEL_9V
