File: hardware/lite/pcb/controller-bus.kicad_sch (KiCad schematic)
At the start: 9 parts, among them J1131 SM04B-SRSS-TB, J1132 UART debug, U1131 TCA9548APWR

Commit message: feat(hardware): use smaller mux, I2C switch, 595 and button packages
The TMUX1511s move to UQFN-16 (RSV), the TCA9548A to VQFN-24 (RGE),
the 74HC595s to TSSOP-16 and the BOOTSEL and RESET buttons to the
Omron B3U, which frees about 300 mm2 of the middle band. The case
button keeps the PTS645.
Parts:
- U1131: value TCA9548APWR -> TCA9548ARGER; footprint Package_SO:TSSOP-24_4.4x7.8mm_P0.65mm -> Package_DFN_QFN:Texas_RGE0024C_VQFN-24-1EP_4x4mm_P0.5mm_EP2.1x2.1mm; symbol Interface_Expansion:TCA9548APWR -> Iasis:TCA9548ARGER; LCSC C130026 -> C555456; MPN TCA9548APWR -> TCA9548ARGER
Connections:
- net 3V3_AON: now also U1131.21 (VCC); no longer U1131.24 (VCC)
- net AON_RESET_N: now also U1131.24 (~{RESET}); no longer U1131.3 (~{RESET})
- net AUX_SCL: now also U1131.17 (SC7); no longer U1131.20 (SC7)
- net AUX_SDA: now also U1131.16 (SD7); no longer U1131.19 (SD7)
- net EXT_SCL: now also U1131.13 (SC5); no longer U1131.16 (SC5)
- net EXT_SDA: now also U1131.12 (SD5); no longer U1131.15 (SD5)
- net GND: now also U1131.18 (A2), U1131.22 (A0), U1131.23 (A1), U1131.9 (GND); no longer U1131.1 (A0), U1131.12 (GND), U1131.2 (A1), U1131.21 (A2)
- net HUB_SCL: now also U1131.15 (SC6); no longer U1131.18 (SC6)
- net HUB_SDA: now also U1131.14 (SD6); no longer U1131.17 (SD6)
- net MCU_I2C_SCL: now also U1131.19 (SCL); no longer U1131.22 (SCL)
- net MCU_I2C_SDA: now also U1131.20 (SDA); no longer U1131.23 (SDA)
- net P1_SCL: now also U1131.2 (SC0); no longer U1131.5 (SC0)
- net P1_SDA: now also U1131.1 (SD0); no longer U1131.4 (SD0)
- net P2_SCL: now also U1131.4 (SC1); no longer U1131.7 (SC1)
- net P2_SDA: now also U1131.3 (SD1); no longer U1131.6 (SD1)
- net P3_SCL: now also U1131.6 (SC2); no longer U1131.9 (SC2)
- net P3_SDA: now also U1131.5 (SD2); no longer U1131.8 (SD2)
- net P4_SCL: now also U1131.8 (SC3); no longer U1131.11 (SC3)
- net P4_SDA: now also U1131.7 (SD3); no longer U1131.10 (SD3)
- net P5_SCL: now also U1131.11 (SC4); no longer U1131.14 (SC4)
- net P5_SDA: now also U1131.10 (SD4); no longer U1131.13 (SD4)
- no-connect marks 0 -> 1
Changed lines of the file:
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@@
 		(color 0 0 0 0)
+	)
+	(no_connect
+		(at 91.44 93.98)
 	)
 	(wire
@@
 	)
 	(symbol
-		(lib_id "Interface_Expansion:TCA9548APWR")
+		(lib_id "Iasis:TCA9548ARGER")
 		(at 101.6 91.44 0)
 		(unit 1)
@@
 			)
 		)
-		(property "Value" "TCA9548APWR"
+		(property "Value" "TCA9548ARGER"
 			(at 92.71 93.98 0)
 			(show_name no)
@@
 			)
 		)
-		(property "Footprint" "Package_SO:TSSOP-24_4.4x7.8mm_P0.65mm"
+		(property "Footprint" "Package_DFN_QFN:Texas_RGE0024C_VQFN-24-1EP_4x4mm_P0.5mm_EP2.1x2.1mm"
 			(at 101.6 91.44 0)
 			(hide yes)
@@
 			)
 		)
-		(property "Description" "Low voltage 8-channel I2C switch with reset, TSSOP-24"
+		(property "Description" "Low voltage 8-channel I2C switch with reset, VQFN-24; exposed pad soldered, no electrical connection"
 			(at 101.6 91.44 0)
 			(hide yes)
@@
 			)
 		)
-		(property "LCSC" "C130026"
+		(property "LCSC" "C555456"
 			(at 101.6 91.44 0)
 			(hide yes)
@@
 			)
 		)
-		(property "MPN" "TCA9548APWR"
+		(property "MPN" "TCA9548ARGER"
 			(at 101.6 91.44 0)
 			(hide yes)
@@
 			)
 		)
+		(pin "22"
+		)
+		(pin "23"
+		)
+		(pin "24"
+		)
 		(pin "1"
 		)
@@
 		(pin "21"
 		)
-		(pin "22"
-		)
-		(pin "23"
-		)
-		(pin "24"
+		(pin "25"
 		)
 		(instances
