File: hardware/lite/pcb/controller-sense.kicad_sch (KiCad schematic)
At the start: 28 parts, among them U1141 TMUX1511PWR, U1142 TMUX1511PWR

Commit message: feat(hardware): use smaller mux, I2C switch, 595 and button packages
The TMUX1511s move to UQFN-16 (RSV), the TCA9548A to VQFN-24 (RGE),
the 74HC595s to TSSOP-16 and the BOOTSEL and RESET buttons to the
Omron B3U, which frees about 300 mm2 of the middle band. The case
button keeps the PTS645.
Parts:
- U1141, U1142: value TMUX1511PWR -> TMUX1511RSVR; footprint Package_SO:TSSOP-14_4.4x5mm_P0.65mm -> Package_DFN_QFN:UQFN-16_1.8x2.6mm_P0.4mm; symbol Iasis:TMUX1511PWR -> Iasis:TMUX1511RSVR; LCSC C2866750 -> C2673275; MPN TMUX1511PWR -> TMUX1511RSVR
Connections:
- net 3V3_AON: now also U1141.16 (VDD), U1142.16 (VDD); no longer U1141.14 (VDD), U1142.14 (VDD)
- net AON_RESET_N: now also U1141.11 (SEL3), U1141.15 (SEL4); no longer U1141.10 (SEL3), U1141.13 (SEL4)
- net GND: now also U1141.8 (GND), U1142.14 (S4), U1142.15 (SEL4); no longer U1141.7 (GND), U1142.12 (S4), U1142.7 (GND)
- net LOCAL_P3_DIV: now also U1141.10 (S3); no longer U1141.9 (S3)
- net LOCAL_P4_DIV: now also U1141.14 (S4); no longer U1141.12 (S4)
- net P3_VBUS_ADC: now also U1141.9 (D3); no longer U1141.8 (D3)
- net P4_VBUS_ADC: now also U1141.13 (D4); no longer U1141.11 (D4)
- no-connect marks 0 -> 4
Changed lines of the file:
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@@
 		(color 0 0 0 0)
 	)
+	(no_connect
+		(at 177.8 160.02)
+	)
+	(no_connect
+		(at 177.8 48.26)
+	)
+	(no_connect
+		(at 177.8 119.38)
+	)
+	(no_connect
+		(at 177.8 88.9)
+	)
 	(wire
 		(pts
@@
 	)
 	(symbol
-		(lib_id "Iasis:TMUX1511PWR")
+		(lib_id "Iasis:TMUX1511RSVR")
 		(at 165.1 139.7 0)
 		(unit 1)
@@
 			)
 		)
-		(property "Value" "TMUX1511PWR"
+		(property "Value" "TMUX1511RSVR"
 			(at 162.56 114.3 0)
 			(show_name no)
@@
 			)
 		)
-		(property "Footprint" "Package_SO:TSSOP-14_4.4x5mm_P0.65mm"
+		(property "Footprint" "Package_DFN_QFN:UQFN-16_1.8x2.6mm_P0.4mm"
 			(at 165.1 139.7 0)
 			(hide yes)
@@
 			)
 		)
-		(property "LCSC" "C2866750"
+		(property "LCSC" "C2673275"
 			(at 165.1 139.7 0)
 			(hide yes)
@@
 			)
 		)
-		(property "MPN" "TMUX1511PWR"
+		(property "MPN" "TMUX1511RSVR"
 			(at 165.1 139.7 0)
 			(hide yes)
@@
 		(pin "6"
 		)
-		(pin "7"
-		)
 		(pin "8"
 		)
@@
 		(pin "11"
 		)
-		(pin "12"
-		)
 		(pin "13"
 		)
 		(pin "14"
 		)
+		(pin "15"
+		)
+		(pin "16"
+		)
+		(pin "7"
+		)
+		(pin "12"
+		)
 		(instances
 			(project "iasis"
@@
 	)
 	(symbol
-		(lib_id "Iasis:TMUX1511PWR")
+		(lib_id "Iasis:TMUX1511RSVR")
 		(at 165.1 68.58 0)
 		(unit 1)
@@
 			)
 		)
-		(property "Value" "TMUX1511PWR"
+		(property "Value" "TMUX1511RSVR"
 			(at 162.56 43.18 0)
 			(show_name no)
@@
 			)
 		)
-		(property "Footprint" "Package_SO:TSSOP-14_4.4x5mm_P0.65mm"
+		(property "Footprint" "Package_DFN_QFN:UQFN-16_1.8x2.6mm_P0.4mm"
 			(at 165.1 68.58 0)
 			(hide yes)
@@
 			)
 		)
-		(property "LCSC" "C2866750"
+		(property "LCSC" "C2673275"
 			(at 165.1 68.58 0)
 			(hide yes)
@@
 			)
 		)
-		(property "MPN" "TMUX1511PWR"
+		(property "MPN" "TMUX1511RSVR"
 			(at 165.1 68.58 0)
 			(hide yes)
@@
 		(pin "6"
 		)
-		(pin "7"
-		)
 		(pin "8"
 		)
@@
 		(pin "11"
 		)
-		(pin "12"
-		)
 		(pin "13"
 		)
 		(pin "14"
 		)
+		(pin "15"
+		)
+		(pin "16"
+		)
+		(pin "7"
+		)
+		(pin "12"
+		)
 		(instances
