File: hardware/lite/pcb/target-charge.kicad_sch (KiCad schematic)
At the start: 37 parts, among them Q1230 2N7002, Q1231 2N7002, Q1232 2N7002, U1230 LMR51450SDRRR, U1231 TPS26600PWPR, U1232 LM4040DIM3X-2.5/NOPB

Commit message: feat(hardware): share brick power across ports and add CM5 link
A connected PD supply now runs the logic through its own buck and feeds
one TPS55288 buck-boost stage per port, so the contract is shared as
5-20 V at up to 5 A per port. The hub's VBUS detect becomes an OR gate,
a host-select mux lets a CM5 side board drive the hub over a 24-pin ZIF
link, and a CM5 variant joins Hub and HubPD.

The board is synced to the schematic and its old routing removed; the
new parts wait below the outline for placement.
Parts:
- removed Q1230, Q1231, Q1232: 2N7002, Package_TO_SOT_SMD:SOT-23, symbol Transistor_FET:2N7002
- removed R1240: 10k, Resistor_SMD:R_0402_1005Metric, symbol Device:R
- removed R1241: 402k 1%, Resistor_SMD:R_0402_1005Metric, symbol Device:R
- removed R1242: 5.49k 1%, Resistor_SMD:R_0402_1005Metric, symbol Device:R
- removed R1243: 39k 1%, Resistor_SMD:R_0402_1005Metric, symbol Device:R
- removed R1244, R1245: 10k 1%, Resistor_SMD:R_0402_1005Metric, symbol Device:R
- removed R1246, R1248: 100k, Resistor_SMD:R_0402_1005Metric, symbol Device:R
- removed R1247: 15k 1%, Resistor_SMD:R_0805_2012Metric, symbol Device:R
- removed TP1231: CHARGE_FAULT_N, TestPoint:TestPoint_Pad_D1.0mm, symbol Connector:TestPoint
- removed U1230: LMR51450SDRRR, Iasis:TI_DRR0012G, symbol Iasis:LMR51450SDRRR
- removed U1231: TPS26600PWPR, Iasis:HTSSOP-16-1EP_4.4x5mm_P0.65mm_EP3.4x5mm_Mask2.66x2.46mm_ThermalVias, symbol Power_Management:TPS26600PWP
- removed U1232: LM4040DIM3X-2.5/NOPB, Package_TO_SOT_SMD:SOT-23, symbol Reference_Voltage:LM4040DBZ-2.5
- added C1240, C1247, C1248: 100n 50V X7R, Capacitor_SMD:C_0402_1005Metric, symbol Device:C
- added C1241, C1242: 100n, Capacitor_SMD:C_0402_1005Metric, symbol Device:C
- added C1243: 10u 16V X5R, Capacitor_SMD:C_0805_2012Metric, symbol Device:C
- added C1244: 10n, Capacitor_SMD:C_0402_1005Metric, symbol Device:C
- added C1245: 4.7n, Capacitor_SMD:C_0402_1005Metric, symbol Device:C
- added C1246: 100p C0G, Capacitor_SMD:C_0402_1005Metric, symbol Device:C
- added Q1230, Q1231: TMGN4060DF, Package_SO:Vishay_PowerPAK_1212-8_Single, symbol Transistor_FET:CSD18543Q3A
- added Q1232, Q1233: SP60N05GNJ, Package_SO:Vishay_PowerPAK_1212-8_Single, symbol Transistor_FET:CSD18543Q3A
- added Q1234: 2N7002, Package_TO_SOT_SMD:SOT-23, symbol Transistor_FET:2N7002
- added R1230: 1, Resistor_SMD:R_0402_1005Metric, symbol Device:R
- added U1230: TPS55288RPMR, Iasis:TI_RPM0026A, symbol Iasis:TPS55288RPMR
- added U1231: LM74502DDFR, Package_TO_SOT_SMD:Texas_DDF0008A_SOT-8_1.6x2.9mm_P0.65mm, symbol Iasis:LM74502DDFR
- C1230, C1231, C1236: value 10u 50V X5R -> 10u 50V X7R; footprint Capacitor_SMD:C_1206_3216Metric -> Capacitor_SMD:C_1210_3225Metric; LCSC C13585 -> C138687; MPN CL31A106KBHNNNE -> CL32B106KBJNNNE
- C1232, C1233, C1238: value 100n 50V X7R -> 10u 50V X7R; footprint Capacitor_SMD:C_0402_1005Metric -> Capacitor_SMD:C_1210_3225Metric; LCSC C307331 -> C138687; MPN CL05B104KB54PNC -> CL32B106KBJNNNE
- C1235: value 10u 50V X5R -> 100n 50V X7R; footprint Capacitor_SMD:C_1206_3216Metric -> Capacitor_SMD:C_0402_1005Metric; LCSC C13585 -> C307331; MPN CL31A106KBHNNNE -> CL05B104KB54PNC
- C1237: value 33p 50V C0G -> 10u 50V X7R; footprint Capacitor_SMD:C_0402_1005Metric -> Capacitor_SMD:C_1210_3225Metric; LCSC C1562 -> C138687; MPN 0402CG330J500NT -> CL32B106KBJNNNE; Manufacturer FH (Guangdong Fenghua Advanced Tech) -> Samsung Electro-Mechanics
- C1239: value 10n 50V X7R -> 10u 50V X7R; footprint Capacitor_SMD:C_0402_1005Metric -> Capacitor_SMD:C_1210_3225Metric; LCSC C15195 -> C138687; MPN CL05B103KB5NNNC -> CL32B106KBJNNNE
- L1230: value 6.8u 12.5A -> 4.7u; footprint Iasis:PSTMAA666460 -> Inductor_SMD:L_Changjiang_FXL1050; LCSC C55172548 -> C54425770; MPN PSTMAA666460-6R8MB -> AAPS1050M4R7A; Manufacturer PROD Tech -> Coilank
- R1231: value 100k 0.1% -> 47k 1%; footprint Resistor_SMD:R_0603_1608Metric -> Resistor_SMD:R_0402_1005Metric; LCSC C122538 -> C25792; MPN RT0603BRD07100KL -> 0402WGF4702TCE; Manufacturer YAGEO -> UNI-ROYAL(Uniroyal Elec)
- R1232, R1236: value 10k 0.1% -> 47k 1%; footprint Resistor_SMD:R_0603_1608Metric -> Resistor_SMD:R_0402_1005Metric; LCSC C95204 -> C25792; MPN RT0603BRD0710KL -> 0402WGF4702TCE; Manufacturer YAGEO -> UNI-ROYAL(Uniroyal Elec)
- R1233: value 10k 0.1% -> 56k 1%; footprint Resistor_SMD:R_0603_1608Metric -> Resistor_SMD:R_0402_1005Metric; LCSC C95204 -> C25796; MPN RT0603BRD0710KL -> 0402WGF5602TCE; Manufacturer YAGEO -> UNI-ROYAL(Uniroyal Elec)
- R1234: value 240k 1% -> 10m 1%; footprint Resistor_SMD:R_0402_1005Metric -> Resistor_SMD:R_1206_3216Metric; LCSC C64043 -> C188070; MPN 0402WGF2403TCE -> RLM12FTCMR010; Manufacturer UNI-ROYAL(Uniroyal Elec) -> RALEC
- R1235: value 10k 0.1% -> 200k 1%; footprint Resistor_SMD:R_0603_1608Metric -> Resistor_SMD:R_0402_1005Metric; LCSC C95204 -> C25764; MPN RT0603BRD0710KL -> 0402WGF2003TCE; Manufacturer YAGEO -> UNI-ROYAL(Uniroyal Elec)
- R1237: value 680k 1% -> 15k 1%; LCSC C4131 -> C25756; MPN 0402WGF6803TCE -> 0402WGF1502TCE
- R1239: value 1k -> 100k; LCSC C11702 -> C25741; MPN 0402WGF1001TCE -> 0402WGF1003TCE
Connections:
- net CHARGE_EN: now also R1239.1, U1231.1 (EN)
- net GND: now also C1233.2, C1237.2, R1231.2, R1232.2, R1236.2, R1239.2, C1240.2, C1243.2, C1244.2, C1245.2, C1246.2, C1248.2, Q1231.1 (S), Q1231.2 (S), Q1231.3 (S), Q1234.2 (S), U1230.10 (AGND), U1230.24 (PGND), U1230.9 (PGND), U1231.2 (GND); no longer R1233.2, R1234.2
- net HV_CHARGE: now also C1233.1, C1235.1, Q1230.5 (D), U1230.3 (VIN)
- net VBUS: now also Q1233.5 (D)
- net OUT_OV: now reaches R1235.2, R1236.1
- net OUT_OV: now also R1237.1, U1231.7 (OV)
- net STAGE_COMP: now reaches R1233.1
- net STAGE_COMP: now also C1246.1, U1230.18 (COMP); no longer R1232.2
- net SW1: now reaches L1230.1
- net SW1: now also C1241.2, Q1230.1 (S), Q1230.2 (S), Q1230.3 (S), Q1231.5 (D), U1230.23 (SW1); no longer C1233.2
- net CONV: now reaches TP1230.1
- net CONV: now also C1234.1, R1234.2, R1235.1, C1247.2, C1248.1, Q1232.5 (D), U1230.13 (ISN), U1231.5 (VS)
- net at R1237.2: now also Q1234.3 (D); no longer R1236.2
- net STAGE_VOUT: now reaches C1239.1
- net STAGE_VOUT: now also C1236.1, C1237.1, C1238.1, R1234.1, C1240.1, U1230.11 (VOUT), U1230.12 (ISP), U1230.26 (VOUT)
- removed net BUCK_VOUT: C1234.1, C1235.1, C1236.1, C1237.1, C1238.1, L1230.2, R1231.1
- removed net FB: R1231.2, R1232.1, R1234.1, R1235.1, R1237.1, R1239.2
- net SEL_9V renamed OV_HIGH
- net OV_HIGH: now also Q1234.1 (G)
- new net: C1247.1, U1231.4 (VCAP)
- new net: C1245.1, R1233.2
- new net: C1242.1, U1230.20 (BOOT2)
- new net: Q1231.4 (G), U1230.1 (DR1L)
- new net: Q1230.4 (G), U1230.2 (DR1H)
- new net: C1241.1, U1230.22 (BOOT1)
- new net 5V_LOGIC: R1230.1
- new net OUT_GATE: Q1232.4 (G), Q1233.4 (G), U1231.6 (GATE)
- new net OUT_SRC: Q1232.1 (S), Q1232.2 (S), Q1232.3 (S), Q1233.1 (S), Q1233.2 (S), Q1233.3 (S), U1231.8 (SRC)
- new net PD_STAGE_EN: U1230.4 (EN_UVLO)
- new net POWER_FAULT_N: U1230.14 (FB_INT)
- new net SCL: U1230.5 (SCL)
- new net SDA: U1230.6 (SDA)
- new net STAGE_DITH: C1244.1, U1230.7 (DITH_SYNC)
- new net STAGE_FSW: R1231.1, U1230.8 (FSW)
- new net STAGE_ILIM: R1232.1, U1230.17 (ILIM)
- new net STAGE_VCC: C1243.1, R1230.2, U1230.19 (VCC)
- new net SW2: C1242.2, L1230.2, U1230.21 (SW2), U1230.25 (SW2)
- no-connect marks 2 -> 3
Other:
- note added: "PD stage — 5 to 20 V, up to 5 A"
- note added: "TPS55288 at I2C 0x75 on the port channel (MODE open: external VCC, PFM). OE defaults off; EN low resets the registers. FSW 47k: 425 kHz. ILIM 47k: 7.0 A average inductor limit. Output limit via 10 mOhm sense, up to 6.35 A by register. Output switch: LM74502 with back-to-back FETs; OV trips at 6.6 V, or 23 V with OV_HIGH set (default off). Hub population: entire sheet DNP."
- note removed: "500 kHz (RT open). EN follows VIN; bucks idle with HV bank on. CHARGE_EN controls the output eFuse only. Join quiet FB ground at U1230."
- note removed: "Feedback: 5.133 V / 9.251 V"
- note removed: "Hub: entire sheet DNP. Charging joins the host branch only at protected connector VBUS."
- note removed: "Nominal OVP divider: 5.83 V / 10.47 V"
- note removed: "Optional target charging — 5 V / 9 V"
- note removed: "RTN/GND/PowerPAD join the ground plane. FLT is separate from host fault: it asserts while off. 2.5 V OVP clamp: measure actual trip levels and fault waveforms."
- note removed: "Start at 5 V / 1 A and 9 V / 1.9 A, subject to input budget. No active-DFU voltage changes. Clear SEL9 with discharge on and eFuse off; wait 3 s (prototype setting), then connect eFuse and verify connector 5 V."
- title: Optional target charging — 5 V / 9 V -> PD stage — 5 to 20 V, up to 5 A
- moved on the sheet: C1234, TP1230

Commit message: refactor(hardware): drop the PD stage output test points
TP1230-TP1630 sat on CONV, which the bulk capacitor's pad already
exposes, and each cost two vias and an inner-layer trace in the stage
cell. Their value still read BUCK_PG from the old buck.
Parts:
- removed TP1230: BUCK_PG, TestPoint:TestPoint_Pad_D1.0mm, symbol Connector:TestPoint
Changed lines of the file:
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@@
-	)
-	(symbol
-		(lib_id "Connector:TestPoint")
-		(at 284.48 60.96 180)
-		(unit 1)
-		(body_style 1)
-		(exclude_from_sim no)
-		(in_bom no)
-		(on_board yes)
-		(in_pos_files no)
-		(dnp no)
-		(property "Reference" "TP1230"
-			(at 284.48 67.818 0)
-			(show_name no)
-			(do_not_autoplace no)
-			(effects
-				(font
-					(size 1.27 1.27)
-				)
-			)
-		)
-		(property "Value" "BUCK_PG"
-			(at 284.48 66.04 0)
-			(show_name no)
-			(do_not_autoplace no)
-			(effects
-				(font
-					(size 1.27 1.27)
-				)
-			)
-		)
-		(property "Footprint" "TestPoint:TestPoint_Pad_D1.0mm"
-			(at 284.48 44.45 0)
-			(hide yes)
-			(show_name no)
-			(do_not_autoplace no)
-			(effects
-				(font
-					(size 1.27 1.27)
-				)
-				(justify left)
-			)
-		)
-		(property "Datasheet" ""
-			(at 284.48 44.45 0)
-			(hide yes)
-			(show_name no)
-			(do_not_autoplace no)
-			(effects
-				(font
-					(size 1.27 1.27)
-				)
-				(justify left)
-			)
-		)
-		(property "Description" ""
-			(at 284.48 44.45 0)
-			(hide yes)
-			(show_name no)
-			(do_not_autoplace no)
-			(effects
-				(font
-					(size 1.27 1.27)
-				)
-				(justify left)
-			)
-		)
-		(property "AssemblyNote" "Copper test pad; no fitted component"
-			(at 284.48 44.45 0)
-			(hide yes)
-			(show_name no)
-			(do_not_autoplace no)
-			(effects
-				(font
-					(size 1.27 1.27)
-				)
-				(justify left)
-			)
-		)
-		(property "Population" "PD"
-			(at 284.48 44.45 0)
-			(hide yes)
-			(show_name no)
-			(do_not_autoplace no)
-			(effects
-				(font
-					(size 1.27 1.27)
-				)
-				(justify left)
-			)
-		)
-		(pin "1"
-		)
-		(instances
-			(project "iasis"
-				(path "/a379403c-5d83-493f-982e-fb5e1b803ee5/eda5d45e-e86d-4d58-83d3-d3aa1de94feb/1980e6d3-fe63-4159-934f-e1343e1cb8bc/7c1e1271-4607-4b20-87e9-40e766ed110f/42bf7062-60f9-4e10-8fdf-2895ab8c3e6f"
-					(reference "TP1330")
-					(unit 1)
-				)
-				(path "/a379403c-5d83-493f-982e-fb5e1b803ee5/eda5d45e-e86d-4d58-83d3-d3aa1de94feb/2661a9c5-45e6-413e-acf1-976df62591a5/7c1e1271-4607-4b20-87e9-40e766ed110f/42bf7062-60f9-4e10-8fdf-2895ab8c3e6f"
-					(reference "TP1430")
-					(unit 1)
-				)
-				(path "/a379403c-5d83-493f-982e-fb5e1b803ee5/eda5d45e-e86d-4d58-83d3-d3aa1de94feb/672b9e1d-749d-4280-bdb9-d44bea0929df/7c1e1271-4607-4b20-87e9-40e766ed110f/42bf7062-60f9-4e10-8fdf-2895ab8c3e6f"
-					(reference "TP1630")
-					(unit 1)
-				)
-				(path "/a379403c-5d83-493f-982e-fb5e1b803ee5/eda5d45e-e86d-4d58-83d3-d3aa1de94feb/973fb476-58e0-4ce2-9f9c-9c93ff84c555/7c1e1271-4607-4b20-87e9-40e766ed110f/42bf7062-60f9-4e10-8fdf-2895ab8c3e6f"
-					(reference "TP1530")
-					(unit 1)
-				)
-				(path "/a379403c-5d83-493f-982e-fb5e1b803ee5/eda5d45e-e86d-4d58-83d3-d3aa1de94feb/acb7f356-15f5-43b4-b29f-4e8b238af2f2/7c1e1271-4607-4b20-87e9-40e766ed110f/42bf7062-60f9-4e10-8fdf-2895ab8c3e6f"
-					(reference "TP1230")
-					(unit 1)
-				)
-			)
-		)
 	)
 	(symbol

Commit message: fix(hardware): join the PD stage analog ground at the VCC capacitor
TPS55288 AGND (pin 10) and the FSW, ILIM, DITH and COMP returns move to a
per-stage STAGE_AGND net. It meets GND only through NT1x30 at the VCC
capacitor's ground terminal, where the datasheet's layout section joins
the two planes, so driver and switching currents stay out of the control
ground.
Parts:
- added NT1330: NetTie_2, NetTie:NetTie-2_SMD_Pad0.5mm, symbol Device:NetTie_2
- renumbered C1230 to C1330, C1231 to C1331, C1232 to C1332, C1233 to C1333, C1234 to C1334, C1235 to C1335, C1236 to C1336, C1237 to C1337, C1238 to C1338, C1239 to C1339, C1240 to C1340, C1241 to C1341, C1242 to C1342, C1243 to C1343, C1244 to C1344, C1245 to C1345, C1246 to C1346, C1247 to C1347, C1248 to C1348, L1230 to L1330, Q1230 to Q1330, Q1231 to Q1331, Q1232 to Q1332, Q1233 to Q1333, Q1234 to Q1334, R1230 to R1330, R1231 to R1331, R1232 to R1332, R1233 to R1333, R1234 to R1334, R1235 to R1335, R1236 to R1336, R1237 to R1337, R1238 to R1338, R1239 to R1339, U1230 to U1330, U1231 to U1331
Connections:
- net GND: now also NT1330.1; no longer C1344.2, C1345.2, C1346.2, R1331.2, R1332.2, U1330.10 (AGND)
- new net STAGE_AGND: C1344.2, C1345.2, C1346.2, NT1330.2, R1331.2, R1332.2, U1330.10 (AGND)
Other:
- moved on the sheet: C1343, R1330
