File: hardware/lite/pcb/power-input.kicad_sch (KiCad schematic)
At the start: 26 parts, among them J1001 USB4105-GF-A-120, Q1001 CSD18543Q3A, Q1002 CSD18543Q3A, U1001 LM74502DDFR, U1002 CH224Q, U1003 TPS26600PWPR

Commit message: feat(hardware): share brick power across ports and add CM5 link
A connected PD supply now runs the logic through its own buck and feeds
one TPS55288 buck-boost stage per port, so the contract is shared as
5-20 V at up to 5 A per port. The hub's VBUS detect becomes an OR gate,
a host-select mux lets a CM5 side board drive the hub over a 24-pin ZIF
link, and a CM5 variant joins Hub and HubPD.

The board is synced to the schematic and its old routing removed; the
new parts wait below the outline for placement.
Parts:
- added C1007: 68u 50V, Capacitor_SMD:CP_Elec_8x10.5, symbol Device:C_Polarized
- added C1008, C1009: 10u 50V X5R, Capacitor_SMD:C_1206_3216Metric, symbol Device:C
- added C1010: 100n 100V X7R, Capacitor_SMD:C_0603_1608Metric, symbol Device:C
- added C1011: 100n, Capacitor_SMD:C_0402_1005Metric, symbol Device:C
- added C1012: 33p C0G, Capacitor_SMD:C_0402_1005Metric, symbol Device:C
- added C1013, C1014, C1015, C1016: 22u 16V X7R, Capacitor_SMD:C_1210_3225Metric, symbol Device:C
- added C1017: 4.7n, Capacitor_SMD:C_0402_1005Metric, symbol Device:C
- added C1018: 100u 35V, Capacitor_SMD:CP_Elec_6.3x7.7, symbol Device:C_Polarized
- added L1004: 6.8u 12.5A, Iasis:PSTMAA666460, symbol Device:L
- added Q1003, Q1004, Q1005: 2N7002, Package_TO_SOT_SMD:SOT-23, symbol Transistor_FET:2N7002
- added R1014, R1021: 47k 1%, Resistor_SMD:R_0402_1005Metric, symbol Device:R
- added R1015, R1020, R1022, R1024: 10k, Resistor_SMD:R_0402_1005Metric, symbol Device:R
- added R1016: 120k 1%, Resistor_SMD:R_0402_1005Metric, symbol Device:R
- added R1017: 22k 1%, Resistor_SMD:R_0402_1005Metric, symbol Device:R
- added R1018, R1025: 1k 1%, Resistor_SMD:R_0402_1005Metric, symbol Device:R
- added R1019, R1023: 39k 1%, Resistor_SMD:R_0402_1005Metric, symbol Device:R
- added R1026, R1029: 100k, Resistor_SMD:R_0402_1005Metric, symbol Device:R
- added R1027: 20k 1%, Resistor_SMD:R_0402_1005Metric, symbol Device:R
- added R1028: 4.7k, Resistor_SMD:R_0402_1005Metric, symbol Device:R
- added U1004: LMR51450SDRRR, Iasis:TI_DRR0012G, symbol Iasis:LMR51450SDRRR
- added U1005: TPS259470ARPWR, Iasis:TI_RPW0010A, symbol Iasis:TPS259470LRPWR
- Q1001, Q1002: value CSD18543Q3A -> SP60N05GNJ; footprint Iasis:TI_CSD18543Q3A -> Package_SO:Vishay_PowerPAK_1212-8_Single; LCSC C840100 -> C22466768; MPN CSD18543Q3A -> SP60N05GNJ; Manufacturer Texas Instruments -> Siliup
- R1008: value 120k 1% -> 6.8k 1%; LCSC C25750 -> C25917; MPN 0402WGF1203TCE -> 0402WGF6801TCE
Connections:
- net GND: now also C1007.2, C1008.2, C1009.2, C1010.2, C1013.2, C1014.2, C1015.2, C1016.2, C1017.2, C1018.2, Q1003.2 (S), Q1005.2 (S), R1015.2, R1017.2, R1020.2, R1022.2, R1024.2, R1025.2, R1028.2, R1029.2, U1004.13 (PGND), U1004.8 (AGND), U1005.8 (GND)
- net HV_CHARGE: now also C1007.1, C1008.1, C1009.1, C1010.1, R1019.1, R1021.1, R1027.1, U1004.10 (VIN), U1004.11 (VIN), U1004.12 (VIN)
- net PD_VBUS_RAW: now also R1014.1
- net PD_INPUT_EN renamed PD_EN
- net PD_EN: now also Q1003.3 (D), R1014.2, R1015.1; no longer R1010.1
- new net: C1012.2, R1018.1
- new net: C1011.2, L1004.1, U1004.1 (SW), U1004.2 (SW), U1004.3 (SW)
- new net: C1011.1, U1004.4 (BOOT)
- new net 5V_LOGIC: C1018.1, R1026.1, U1005.6 (OUT)
- new net AUXOFF: Q1004.1 (G), R1026.2, U1005.3 (AUXOFF)
- new net EXT_VBUS: Q1004.3 (D)
- new net LOGIC_5V2: C1012.1, C1013.1, C1014.1, C1015.1, C1016.1, L1004.2, R1016.1, R1023.1, U1005.5 (IN)
- new net LOGIC_BUCK_EN: R1019.2, R1020.1, U1004.9 (EN)
- new net LOGIC_FB: R1016.2, R1017.1, R1018.2, U1004.7 (FB)
- new net LOGIC_OVLO: Q1004.2 (S)
- new net LOGIC_PRI_DVDT: C1017.1, U1005.7 (DVDT)
- new net LOGIC_PRI_EN: R1021.2, R1022.1, U1005.1 (EN_UVLO)
- new net LOGIC_PRI_ILM: R1025.1, U1005.9 (ILM)
- new net LOGIC_PRI_OVLO: R1023.2, R1024.1, U1005.2 (OVLO)
- new net PD_INPUT_OFF: Q1003.1 (G), R1010.1
- new net PD_STAGE_EN: Q1005.3 (D), R1027.2, R1028.1
- new net PORT_STAGES_OFF: Q1005.1 (G), R1029.1
- no-connect marks 11 -> 15
Other:
- note added: "Brick input and logic child"
- note added: "CFG1 6.8k requests 9 V by default, so a brick alone starts the board; firmware then requests 28 V EPR or 20 V over I2C."
- note removed: "CFG1 selects 20 V default. Request 28 V only after source/cable capability checks. I2C mux channel 7. VHV and VBUS share a filtered, protected supply. CC pins remain connected to raw CC. Input transients and CC shorts need bench qualification."
- note removed: "Optional USB-C charging input"
- title: Optional USB-C charging input -> Brick input and logic child
- moved on the sheet: R1010

Commit message: feat(hardware): drop the tall input cans and the X5R input ceramics
The CH224 supply's 68 uF can becomes a 10 uF X7R ceramic and the bus
bulk a 33 uF 6.3 x 7.7 mm hybrid, so no part stands taller than the
port bulk caps and the case roof can come down by about 4 mm. The
logic child and CH224 ceramics move from X5R 1206 to the stages'
X7R 1210, which keeps about 4 uF each at 28 V instead of 1.2 uF.
Parts:
- removed C1002: 68u 50V, Capacitor_SMD:CP_Elec_8x10.5, symbol Device:C_Polarized
- added C1002: 10u 50V X7R, Capacitor_SMD:C_1210_3225Metric, symbol Device:C
- C1003, C1008, C1009: value 10u 50V X5R -> 10u 50V X7R; footprint Capacitor_SMD:C_1206_3216Metric -> Capacitor_SMD:C_1210_3225Metric; LCSC C13585 -> C138687; MPN CL31A106KBHNNNE -> CL32B106KBJNNNE
- C1007: value 68u 50V -> 33u 50V; footprint Capacitor_SMD:CP_Elec_8x10.5 -> Capacitor_SMD:CP_Elec_6.3x7.7; LCSC C178645 -> C178637; MPN EEHZC1H680P -> EEHZA1H330XP
Connections:
- net GND: now also C1002.2
- net at R1007.1, U1003.15 (OUT), U1003.16 (OUT): now also C1002.1

Commit message: feat(pcb): route core and power distribution
Parts:
- C1012: Manufacturer Samsung Electro-Mechanics -> FH (Guangdong Fenghua Advanced Tech)
Changed lines of the file:
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@@
 			)
 		)
-		(property "Manufacturer" "Samsung Electro-Mechanics"
+		(property "Manufacturer" "FH (Guangdong Fenghua Advanced Tech)"
 			(at 167.64 266.7 0)
 			(hide yes)

Commit message: fix: lower logic supply overvoltage cutoff
Parts:
- R1023: value 39k 1% -> 36.5k 1%; LCSC C25783 -> C25887; MPN 0402WGF3902TCE -> 0402WGF3652TCE
Changed lines of the file:
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@@
 			)
 		)
-		(property "Value" "39k 1%"
+		(property "Value" "36.5k 1%"
 			(at 251.46 311.15 0)
 			(show_name no)
@@
 			)
 		)
-		(property "Datasheet" "https://www.lcsc.com/datasheet/lcsc_datasheet_2206010100_UNI-ROYAL-Uniroyal-Elec-0402WGF3902TCE_C25783.pdf"
+		(property "Datasheet" "https://www.lcsc.com/datasheet/lcsc_datasheet_2206010045_UNI-ROYAL-Uniroyal-Elec-0402WGF3652TCE_C25887.pdf"
 			(at 248.92 311.15 0)
 			(hide yes)
@@
 			)
 		)
-		(property "LCSC" "C25783"
+		(property "LCSC" "C25887"
 			(at 248.92 311.15 0)
 			(hide yes)
@@
 			)
 		)
-		(property "MPN" "0402WGF3902TCE"
+		(property "MPN" "0402WGF3652TCE"
 			(at 248.92 311.15 0)
 			(hide yes)
