File: hardware/boards/iasis/iasis.kicad_pcb (KiCad board)
At the start: 6 copper layers, 133 x 102 mm, 718 parts, among them J1001 USB4105-GF-A-120, J1101 SWD debug, J1131 SM04B-SRSS-TB, J1132 UART debug, J2001 05A20L24P, J401 1054500101, J501 1054500101, J601 1054500101, J701 1054500101, J801 1054500101, J901 1054500101, Q1001 SP60N05GNJ, Q1002 SP60N05GNJ, Q1003 2N7002, Q1004 2N7002, Q1005 2N7002, Q1221 2N7002, Q1230 TMGN4060DF, Q1231 TMGN4060DF, Q1232 SP60N05GNJ, Q1233 SP60N05GNJ, Q1234 2N7002, Q1321 2N7002, Q1330 TMGN4060DF, Q1331 TMGN4060DF, Q1332 SP60N05GNJ, Q1333 SP60N05GNJ, Q1334 2N7002, Q1421 2N7002, Q1430 TMGN4060DF, Q1431 TMGN4060DF, Q1432 SP60N05GNJ, Q1433 SP60N05GNJ, Q1434 2N7002, Q1521 2N7002, Q1530 TMGN4060DF, Q1531 TMGN4060DF, Q1532 SP60N05GNJ, Q1533 SP60N05GNJ, Q1534 2N7002, Q1621 2N7002, Q1630 TMGN4060DF, Q1631 TMGN4060DF, Q1632 SP60N05GNJ, Q1633 SP60N05GNJ, Q1634 2N7002, Q1911 2N7002, Q1912 2N7002, Q901 2N7002, Q902 2N7002, SW1101 B3U-1000P, SW1102 B3U-1000P, SW1171 PTS645SL50SMTR92LFS, U1001 LM74502DDFR, U1002 CH224Q, U1003 TPS26600PWPR, U1004 LMR51450SDRRR, U1005 TPS259470ARPWR, U1040 AP3441SHE-7B, U1060 AP3441SHE-7B, U1080 TPS3808G33DBVR, U1101 RP2354B, U1131 TCA9548ARGER, U1141 TMUX1511RSVR, U1142 TMUX1511RSVR, U1171 SN74AHCT1G125DBVR, U1172 TCA6408ARGTR, U1181 74HC595PW, U1182 74HC595PW, U1202 TPS259470ARPWR, U1203 74LVC2G08DC-Q100H, U1230 TPS55288RPMR, U1231 LM74502DDFR, U1302 TPS259470ARPWR, U1303 74LVC2G08DC-Q100H, U1330 TPS55288RPMR, U1331 LM74502DDFR, U1402 TPS259470ARPWR, U1403 74LVC2G08DC-Q100H, U1430 TPS55288RPMR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

Commit message: fix(pcb): simplify routing and support placement
Parts:
- moved C903 7.08 mm to (96.4, 73.9), turned to -90 degrees
- moved R1171 5.59 mm to (176.1, 148.8), turned to -90 degrees
- moved C1171 2.20 mm to (176.1, 143.0), turned to 90 degrees
- moved C1175 0.64 mm to (81.8, 148.8), turned to 90 degrees
- moved C1176 0.64 mm to (105.8, 148.8), turned to 90 degrees
- moved C1170 0.64 mm to (178.8, 148.8), turned to 90 degrees
- moved C1177 0.64 mm to (129.8, 148.8), turned to 90 degrees
- moved C1178 0.64 mm to (153.8, 148.8), turned to 90 degrees
Routing:
- net /Indicators and confirmation/LED_DIN0: track 11.5 -> 2.07 mm
- net EXT_SCL: track 78.2 -> 68.9 mm
- net P3_SCL: track 158.5 -> 149.8 mm
- net /Host port/VBIAS: track 10.9 -> 2.61 mm, vias 2 -> 0
- net P5_OV_HIGH: track 142.7 -> 135.0 mm
- net P3_SDA: track 150.3 -> 144.1 mm
- net PD_STAGE_EN: track 175.6 -> 169.5 mm
- net INPUT_PROTECT_FAULT_N: track 130.1 -> 124.1 mm, vias 12 -> 11
- net P2_CHARGE_EN_REQ: track 159.1 -> 154.0 mm
- net /Indicators and confirmation/LED_DRIVE: track 6.13 -> 1.34 mm
- net /Brick input and logic child/CH_SUPPLY: track 14.7 -> 10.1 mm
- net P2_SDA: track 259.0 -> 254.9 mm
- net P4_SCL: track 137.1 -> 133.3 mm
- net P2_SCL: track 219.3 -> 215.5 mm
- net P5_SCL: track 104.1 -> 100.7 mm
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