File: hardware/boards/iasis/side-link.kicad_sch (KiCad schematic)
At the start: 10 parts, among them J2001 05A20L24P, U2001 TPS26600PWPR

Commit message: feat(iasis): reroute the board for the case and the FH12 side link
The side link J2001 is a Hirose FH12-24S-0.5SVA(54). Its contact-side row escapes between the
inboard lands under a 0.12 mm DRU rule. The RP2354's signal nets and those of the I2C switch U1131
use the MCU_IO class (0.1 mm tracks and clearance), so the 0.4 mm QFN fans out on 0.45 mm vias.

Mounting holes H5 and H6 and SW1171 sit where the case needs them. Every net is routed, with the
slow signals on 45-degree runs across F.Cu, B.Cu, In2 and In3. DRC, schematic parity and ERC pass.
The case previews show this board.
Parts:
- J2001: value 05A20L24P -> FH12-24S-0.5SVA(54); footprint Iasis:HanElectricity_05A20L24P -> Iasis:Hirose_FH12-24S-0.5SVA_1x24-1MP_P0.50mm_Vertical; LCSC C5362158 -> C3169218; MPN 05A20L24P -> FH12-24S-0.5SVA(54); Manufacturer HanElectricity -> Hirose
Changed lines of the file:
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@@
 			)
 		)
-		(property "Value" "05A20L24P"
+		(property "Value" "FH12-24S-0.5SVA(54)"
 			(at 238.76 101.6 0)
 			(show_name no)
@@
 			)
 		)
-		(property "Footprint" "Iasis:HanElectricity_05A20L24P"
+		(property "Footprint" "Iasis:Hirose_FH12-24S-0.5SVA_1x24-1MP_P0.50mm_Vertical"
 			(at 236.22 99.06 0)
 			(hide yes)
@@
 			)
 		)
-		(property "LCSC" "C5362158"
+		(property "LCSC" "C3169218"
 			(at 236.22 99.06 0)
 			(hide yes)
@@
 			)
 		)
-		(property "MPN" "05A20L24P"
+		(property "MPN" "FH12-24S-0.5SVA(54)"
 			(at 236.22 99.06 0)
 			(hide yes)
@@
 			)
 		)
-		(property "Manufacturer" "HanElectricity"
+		(property "Manufacturer" "Hirose"
 			(at 236.22 99.06 0)
 			(hide yes)

Commit message: feat(hardware): use stocked CM5 headers
Parts:
- C2001, C2002, C2003, R2001, R2002, R2003, R2004, R2005, U2001: Population CM5 -> HubPD,CM5
- J2001: value FH12-24S-0.5SVA(54) -> KH-2FH90-2X10P-H6.35; footprint Iasis:Hirose_FH12-24S-0.5SVA_1x24-1MP_P0.50mm_Vertical -> Connector_PinSocket_2.00mm:PinSocket_2x10_P2.00mm_Horizontal; symbol Connector_Generic_MountingPin:Conn_01x24_MountingPin -> Connector_Generic:Conn_01x20; LCSC C3169218 -> C49424687; MPN FH12-24S-0.5SVA(54) -> KH-2FH90-2X10P-H6.35; Manufacturer Hirose -> Kinghelm; Population CM5 -> HubPD,CM5
Connections:
- net CM5_HOST: now also J2001.8 (Pin_8); no longer J2001.11 (Pin_11)
- net GND: now also J2001.12 (Pin_12), J2001.2 (Pin_2), J2001.20 (Pin_20), J2001.6 (Pin_6); no longer J2001.14 (Pin_14), J2001.21 (Pin_21), J2001.22 (Pin_22), J2001.23 (Pin_23), J2001.24 (Pin_24), J2001.MP (MountPin)
- net SIDE_BUS: no longer J2001.16 (Pin_16), J2001.18 (Pin_18), J2001.20 (Pin_20)
- net SIDE_D_N: now also J2001.16 (Pin_16); no longer J2001.9 (Pin_9)
- net SIDE_D_P: now also J2001.18 (Pin_18); no longer J2001.8 (Pin_8)
- net SIDE_PRESENT_N: now also J2001.14 (Pin_14); no longer J2001.12 (Pin_12)
- net SIDE_RX_N: now also J2001.11 (Pin_11); no longer J2001.6 (Pin_6)
- net SIDE_RX_P: now also J2001.9 (Pin_9); no longer J2001.5 (Pin_5)
- net SIDE_TX_N: now also J2001.5 (Pin_5); no longer J2001.3 (Pin_3)
- net SIDE_TX_P: now also J2001.3 (Pin_3); no longer J2001.2 (Pin_2)
Other:
- note added: "HubPD and CM5: side link fitted; Hub: sheet DNP. SIDE_POWER_EN enables the feed after firmware reserves 32 W on a 20 V or higher contract. ILIM 5.6k: 2.14 A. Three SIDE_BUS contacts; nine grounds. Mate only with power disconnected."
- note added: "Side link — CM5 board feed and socket"
- note removed: "CM5 build only (Hub and HubPD: sheet DNP). SIDE_POWER_EN (GPIO22) enables the feed after firmware reserves 32 W on a 20 V or higher contract. ILIM 5.6k: 2.14 A. Flex: custom two-layer, 90 Ohm pairs, about 20 mm."
- note removed: "Side link — CM5 board feed and ZIF"
- title: Side link — CM5 board feed and ZIF -> Side link — CM5 board feed and socket
