File: hardware/boards/iasis/side-link.kicad_sch (KiCad schematic)
At the start: 10 parts, among them J2001 KH-2FH90-2X10P-H6.35, U2001 TPS26600PWPR

Commit message: fix(hardware): replace side-link socket with C19268939
Update J2001 supplier fields, mechanical model, outlines, placement correction and preview while retaining its pad pattern and copper.
Parts:
- J2001: value KH-2FH90-2X10P-H6.35 -> XDM200-2-10-W-6.35-G0; LCSC C49424687 -> C19268939; MPN KH-2FH90-2X10P-H6.35 -> XDM200-2-10-W-6.35-G0; Manufacturer Kinghelm -> chxunda
Changed lines of the file:
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@@
 			)
 		)
-		(property "Value" "KH-2FH90-2X10P-H6.35"
+		(property "Value" "XDM200-2-10-W-6.35-G0"
 			(at 238.76 101.6 0)
 			(show_name no)
@@
 			)
 		)
-		(property "Datasheet" "https://www.lcsc.com/datasheet/C49424687.pdf"
+		(property "Datasheet" "https://www.lcsc.com/datasheet/C19268939.pdf"
 			(at 236.22 99.06 0)
 			(hide yes)
@@
 			)
 		)
-		(property "LCSC" "C49424687"
+		(property "LCSC" "C19268939"
 			(at 236.22 99.06 0)
 			(hide yes)
@@
 			)
 		)
-		(property "MPN" "KH-2FH90-2X10P-H6.35"
+		(property "MPN" "XDM200-2-10-W-6.35-G0"
 			(at 236.22 99.06 0)
 			(hide yes)
@@
 			)
 		)
-		(property "Manufacturer" "Kinghelm"
+		(property "Manufacturer" "chxunda"
 			(at 236.22 99.06 0)
 			(hide yes)
