File: hardware/boards/iasis/controller-bus.kicad_sch (KiCad schematic)
At the start: 9 parts, among them J1131 SM04B-SRSS-TB, J1132 UART debug, U1131 TCA9548ARGER

Commit message: feat(hardware): add independent mux reset
Parts:
- added C1132: 100n, Capacitor_SMD:C_0402_1005Metric, symbol Device:C
- added R1133: 10k, Resistor_SMD:R_0402_1005Metric, symbol Device:R
- added U1132: SN74AUP1G08DCKR, Package_TO_SOT_SMD:SOT-353_SC-70-5, symbol 74xGxx:74AUP1G08
- J1132: value UART debug -> UART TX debug
- R1135: value 10k -> 4.7k; LCSC C25744 -> C25900; MPN 0402WGF1002TCE -> 0402WGF4701TCE
Connections:
- net 3V3_AON: now also C1132.1, R1133.1, U1132.5 (VCC); no longer R1135.1
- net AON_RESET_N: now also U1132.1; no longer U1131.24 (~{RESET})
- net GND: now also R1135.2, C1132.2, U1132.3 (GND)
- net MCU_UART_RX: no longer names the net of J1132.1 (Pin_1)
- net MCU_UART_RX: no longer R1135.2
- new net MUX_RUN: R1135.1, U1132.2
- new net TCA_RESET_N: R1133.2, U1131.24 (~{RESET}), U1132.4
- no-connect marks 1 -> 2
Other:
- note added: "J1132 is the 3.3 V UART log output: NC / GND / TX solder pads. Power the board from its host port before using UART; do not connect an adapter supply."
- note added: "MUX_RUN is held low until firmware releases the mux. Physical RESET also deselects every mux channel. Expander reset remains independent on GPIO32."
- note removed: "J1132 is the 3.3 V UART debug port: RX / GND / TX solder pads. Power the board from its host port before using UART; do not connect an adapter supply."
- moved on the sheet: R1135
