File: hardware/boards/cm5/accessory-port.kicad_sch (KiCad schematic)
At the start: 20 parts, among them J401 1054500101, Q401 2N7002, U401 HD3SS3220RNHR, U402 AP22652W6-7, U403 TPD4E02B04DQAR, U404 TPD4E02B04DQAR, U405 TPD4E05U06DQAR

Commit message: feat(cm5): add the status light and short M.2 standoffs, space the rear ports
The side board grows to the main board's 102 mm depth, so the status light sits at the enclosure's front wall and the 2280 standoff clears the rear strip. RJ45, accessory and service USB-C now have even gaps with H4 between the USB-Cs and nRPIBOOT beside the service port. The status light is the main board's SK6812SIDE-A behind an SN74AHCT1G125 on GPIO10; H702 and H703 take 2230 and 2242 drives. The accessory ESD follows the main board's port cell, with TX1/TX2 polarity swapped at the receptacle as there.
Connections:
- net TX1_N: now also J401.A2 (TX1+); no longer J401.A3 (TX1-)
- net TX1_P: now also J401.A3 (TX1-); no longer J401.A2 (TX1+)
- net TX2_N: now also J401.B2 (TX2+); no longer J401.B3 (TX2-)
- net TX2_P: now also J401.B3 (TX2-); no longer J401.B2 (TX2+)
Other:
- note added: "U401 runs as a DFP: PORT high, ADDR open (GPIO mode), CURRENT_MODE 499k advertises 1.5 A. ID goes low when a sink attaches and turns on U402, which limits VBUS to 1.7 A. VBUS_EN low holds CC_EN_N high, so the port stays off until the CM5 enables USB power. U401 sources VCONN from 5V; C401 is its bulk capacitor (10 µF minimum). TX1 and TX2 reach the receptacle with swapped polarity, as on the main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"
- note removed: "U401 runs as a DFP: PORT high, ADDR open (GPIO mode), CURRENT_MODE 499k advertises 1.5 A. ID goes low when a sink attaches and turns on U402, which limits VBUS to 1.7 A. VBUS_EN low holds CC_EN_N high, so the port stays off until the CM5 enables USB power. U401 sources VCONN from 5V; C401 is its bulk capacitor (10 µF minimum)."
Changed lines of the file:
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@@
 (label "RX1_N" (at 307.34 121.92 180) (effects (font (size 1.27 1.27)) (justify right bottom)))
 (label "RX1_P" (at 307.34 124.46 180) (effects (font (size 1.27 1.27)) (justify right bottom)))
-(label "TX1_N" (at 307.34 129.54 180) (effects (font (size 1.27 1.27)) (justify right bottom)))
-(label "TX1_P" (at 307.34 132.08 180) (effects (font (size 1.27 1.27)) (justify right bottom)))
+(label "TX1_P" (at 307.34 129.54 180) (effects (font (size 1.27 1.27)) (justify right bottom)))
+(label "TX1_N" (at 307.34 132.08 180) (effects (font (size 1.27 1.27)) (justify right bottom)))
 (label "RX2_N" (at 307.34 137.16 180) (effects (font (size 1.27 1.27)) (justify right bottom)))
 (label "RX2_P" (at 307.34 139.7 180) (effects (font (size 1.27 1.27)) (justify right bottom)))
-(label "TX2_N" (at 307.34 144.78 180) (effects (font (size 1.27 1.27)) (justify right bottom)))
-(label "TX2_P" (at 307.34 147.32 180) (effects (font (size 1.27 1.27)) (justify right bottom)))
+(label "TX2_P" (at 307.34 144.78 180) (effects (font (size 1.27 1.27)) (justify right bottom)))
+(label "TX2_N" (at 307.34 147.32 180) (effects (font (size 1.27 1.27)) (justify right bottom)))
 (label "CC1" (at 248.92 101.6 0) (effects (font (size 1.27 1.27)) (justify left bottom)))
 (label "CC2" (at 248.92 104.14 0) (effects (font (size 1.27 1.27)) (justify left bottom)))
@@
 (text "SuperSpeed ESD" (exclude_from_sim no) (at 187.96 160.02 0) (effects (font (size 1.778 1.778) (bold yes)) (justify left top)))
 (text "Route through both pads" (exclude_from_sim no) (at 124.46 205.74 0) (effects (font (size 1.27 1.27)) (justify left top)))
-(text "U401 runs as a DFP: PORT high, ADDR open (GPIO mode), CURRENT_MODE 499k advertises 1.5 A.\nID goes low when a sink attaches and turns on U402, which limits VBUS to 1.7 A.\nVBUS_EN low holds CC_EN_N high, so the port stays off until the CM5 enables USB power.\nU401 sources VCONN from 5V; C401 is its bulk capacitor (10 µF minimum)." (exclude_from_sim no) (at 25.4 228.6 0) (effects (font (size 1.27 1.27)) (justify left top)))
+(text "U401 runs as a DFP: PORT high, ADDR open (GPIO mode), CURRENT_MODE 499k advertises 1.5 A.\nID goes low when a sink attaches and turns on U402, which limits VBUS to 1.7 A.\nVBUS_EN low holds CC_EN_N high, so the port stays off until the CM5 enables USB power.\nU401 sources VCONN from 5V; C401 is its bulk capacitor (10 µF minimum).\nTX1 and TX2 reach the receptacle with swapped polarity, as on the main board; USB 3 receivers correct it." (exclude_from_sim no) (at 25.4 228.6 0) (effects (font (size 1.27 1.27)) (justify left top)))
 (embedded_fonts no)
 )
