File: hardware/boards/cm5/nvme.kicad_sch (KiCad schematic)
At the start: 15 parts, among them J701 1-2199230-5, U701 AP3441SHE-7B

Commit message: feat(cm5): add the status light and short M.2 standoffs, space the rear ports
The side board grows to the main board's 102 mm depth, so the status light sits at the enclosure's front wall and the 2280 standoff clears the rear strip. RJ45, accessory and service USB-C now have even gaps with H4 between the USB-Cs and nRPIBOOT beside the service port. The status light is the main board's SK6812SIDE-A behind an SN74AHCT1G125 on GPIO10; H702 and H703 take 2230 and 2242 drives. The accessory ESD follows the main board's port cell, with TX1/TX2 polarity swapped at the receptacle as there.
Parts:
- added H702, H703: 9774025243R, Mounting_Wuerth:Mounting_Wuerth_WA-SMSI-M2_H2.5mm_9774025243, symbol Mechanical:MountingHole_Pad
Connections:
- net GND: now also H702.1, H703.1
Other:
- note added: "PCIE_PWR_EN switches the socket supply; R703 keeps it off until the CM5 drives it. Lane 0 runs at spec polarity; standoffs H701, H702 and H703 take 2280, 2230 and 2242 drives."
- note removed: "PCIE_PWR_EN switches the socket supply; R703 keeps it off until the CM5 drives it. Lane 0 runs at spec polarity; H701 is the drive standoff."
Changed lines of the file:
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@@
+		)
+	)
+(symbol
+		(lib_id "Mechanical:MountingHole_Pad")
+		(at 370.84 134.62 0)
+		(unit 1)
+		(body_style 1)
+		(exclude_from_sim no)
+		(in_bom yes)
+		(on_board yes)
+		(in_pos_files yes)
+		(dnp no)
+		(property "Reference" "H702"
+			(at 373.38 132.08 0)
+			(show_name no)
+			(do_not_autoplace no)
+			(effects (font (size 1.27 1.27)) (justify left))
+		)
+		(property "Value" "9774025243R"
+			(at 373.38 134.62 0)
+			(show_name no)
+			(do_not_autoplace no)
+			(effects (font (size 1.27 1.27)) (justify left))
+		)
+		(property "Footprint" "Mounting_Wuerth:Mounting_Wuerth_WA-SMSI-M2_H2.5mm_9774025243"
+			(at 370.84 134.62 0)
+			(hide yes)
+			(show_name no)
+			(do_not_autoplace no)
+			(effects
+				(font
+					(size 1.27 1.27)
+				)
+			)
+		)
+		(property "Datasheet" "https://www.we-online.com/components/products/datasheet/9774025243R.pdf"
+			(at 370.84 134.62 0)
+			(hide yes)
+			(show_name no)
+			(do_not_autoplace no)
+			(effects
+				(font
+					(size 1.27 1.27)
+				)
+			)
+		)
+		(property "Description" "Mounting Hole with connection"
+			(at 370.84 134.62 0)
+			(hide yes)
+			(show_name no)
+			(do_not_autoplace no)
+			(effects
+				(font
+					(size 1.27 1.27)
+				)
+			)
+		)
+		(property "LCSC" "C22431115"
+			(at 370.84 134.62 0)
+			(hide yes)
+			(show_name no)
+			(do_not_autoplace no)
+			(effects
+				(font
+					(size 1.27 1.27)
+				)
+			)
+		)
+		(property "MPN" "9774025243R"
+			(at 370.84 134.62 0)
+			(hide yes)
+			(show_name no)
+			(do_not_autoplace no)
+			(effects
+				(font
+					(size 1.27 1.27)
+				)
+			)
+		)
+		(property "Manufacturer" "Wurth Elektronik"
+			(at 370.84 134.62 0)
+			(hide yes)
+			(show_name no)
+			(do_not_autoplace no)
+			(effects
+				(font
+					(size 1.27 1.27)
+				)
+			)
+		)
+		(pin "1"
+		)
+		(instances
+			(project "cm5"
+				(path "/6a022b51-582b-478a-88ab-528b7c0cb8e3/cdfcfd2c-3c7a-4183-aa6d-700ec5c19d6e"
+					(reference "H702")
+					(unit 1)
+				)
+			)
+		)
+	)
+(symbol
+		(lib_id "Mechanical:MountingHole_Pad")
+		(at 370.84 152.4 0)
+		(unit 1)
+		(body_style 1)
+		(exclude_from_sim no)
+		(in_bom yes)
+		(on_board yes)
+		(in_pos_files yes)
+		(dnp no)
+		(property "Reference" "H703"
+			(at 373.38 149.86 0)
+			(show_name no)
+			(do_not_autoplace no)
+			(effects (font (size 1.27 1.27)) (justify left))
+		)
+		(property "Value" "9774025243R"
+			(at 373.38 152.4 0)
+			(show_name no)
+			(do_not_autoplace no)
+			(effects (font (size 1.27 1.27)) (justify left))
+		)
+		(property "Footprint" "Mounting_Wuerth:Mounting_Wuerth_WA-SMSI-M2_H2.5mm_9774025243"
+			(at 370.84 152.4 0)
+			(hide yes)
+			(show_name no)
+			(do_not_autoplace no)
+			(effects
+				(font
+					(size 1.27 1.27)
+				)
+			)
+		)
+		(property "Datasheet" "https://www.we-online.com/components/products/datasheet/9774025243R.pdf"
+			(at 370.84 152.4 0)
+			(hide yes)
+			(show_name no)
+			(do_not_autoplace no)
+			(effects
+				(font
+					(size 1.27 1.27)
+				)
+			)
+		)
+		(property "Description" "Mounting Hole with connection"
+			(at 370.84 152.4 0)
+			(hide yes)
+			(show_name no)
+			(do_not_autoplace no)
+			(effects
+				(font
+					(size 1.27 1.27)
+				)
+			)
+		)
+		(property "LCSC" "C22431115"
+			(at 370.84 152.4 0)
+			(hide yes)
+			(show_name no)
+			(do_not_autoplace no)
+			(effects
+				(font
+					(size 1.27 1.27)
+				)
+			)
+		)
+		(property "MPN" "9774025243R"
+			(at 370.84 152.4 0)
+			(hide yes)
+			(show_name no)
+			(do_not_autoplace no)
+			(effects
+				(font
+					(size 1.27 1.27)
+				)
+			)
+		)
+		(property "Manufacturer" "Wurth Elektronik"
+			(at 370.84 152.4 0)
+			(hide yes)
+			(show_name no)
+			(do_not_autoplace no)
+			(effects
+				(font
+					(size 1.27 1.27)
+				)
+			)
+		)
+		(pin "1"
+		)
+		(instances
+			(project "cm5"
+				(path "/6a022b51-582b-478a-88ab-528b7c0cb8e3/cdfcfd2c-3c7a-4183-aa6d-700ec5c19d6e"
+					(reference "H703")
+					(unit 1)
+				)
+			)
 		)
 	)
@@
 (symbol (lib_id "power:GND") (at 335.28 203.2 0) (unit 1) (body_style 1) (exclude_from_sim no) (in_bom yes) (on_board yes) (in_pos_files yes) (dnp no) (property "Reference" "#PWR5032015" (at 335.28 203.2 0) (hide yes) (effects (font (size 1.27 1.27)))) (property "Value" "GND" (at 335.28 207.01 0) (effects (font (size 1.27 1.27)))) (property "Footprint" "" (at 335.28 203.2 0) (hide yes) (effects (font (size 1.27 1.27)))) (property "Datasheet" "" (at 335.28 203.2 0) (hide yes) (effects (font (size 1.27 1.27)))) (pin "1") (instances (project "cm5" (path "/6a022b51-582b-478a-88ab-528b7c0cb8e3/cdfcfd2c-3c7a-4183-aa6d-700ec5c19d6e" (reference "#PWR5032015") (unit 1)))))
 (symbol (lib_id "power:GND") (at 370.84 121.92 0) (unit 1) (body_style 1) (exclude_from_sim no) (in_bom yes) (on_board yes) (in_pos_files yes) (dnp no) (property "Reference" "#PWR5032016" (at 370.84 121.92 0) (hide yes) (effects (font (size 1.27 1.27)))) (property "Value" "GND" (at 370.84 125.73 0) (effects (font (size 1.27 1.27)))) (property "Footprint" "" (at 370.84 121.92 0) (hide yes) (effects (font (size 1.27 1.27)))) (property "Datasheet" "" (at 370.84 121.92 0) (hide yes) (effects (font (size 1.27 1.27)))) (pin "1") (instances (project "cm5" (path "/6a022b51-582b-478a-88ab-528b7c0cb8e3/cdfcfd2c-3c7a-4183-aa6d-700ec5c19d6e" (reference "#PWR5032016") (unit 1)))))
+(symbol (lib_id "power:GND") (at 370.84 139.7 0) (unit 1) (body_style 1) (exclude_from_sim no) (in_bom yes) (on_board yes) (in_pos_files yes) (dnp no) (property "Reference" "#PWR5032017" (at 370.84 139.7 0) (hide yes) (effects (font (size 1.27 1.27)))) (property "Value" "GND" (at 370.84 143.51 0) (effects (font (size 1.27 1.27)))) (property "Footprint" "" (at 370.84 139.7 0) (hide yes) (effects (font (size 1.27 1.27)))) (property "Datasheet" "" (at 370.84 139.7 0) (hide yes) (effects (font (size 1.27 1.27)))) (pin "1") (instances (project "cm5" (path "/6a022b51-582b-478a-88ab-528b7c0cb8e3/cdfcfd2c-3c7a-4183-aa6d-700ec5c19d6e" (reference "#PWR5032017") (unit 1)))))
+(symbol (lib_id "power:GND") (at 370.84 157.48 0) (unit 1) (body_style 1) (exclude_from_sim no) (in_bom yes) (on_board yes) (in_pos_files yes) (dnp no) (property "Reference" "#PWR5032018" (at 370.84 157.48 0) (hide yes) (effects (font (size 1.27 1.27)))) (property "Value" "GND" (at 370.84 161.29 0) (effects (font (size 1.27 1.27)))) (property "Footprint" "" (at 370.84 157.48 0) (hide yes) (effects (font (size 1.27 1.27)))) (property "Datasheet" "" (at 370.84 157.48 0) (hide yes) (effects (font (size 1.27 1.27)))) (pin "1") (instances (project "cm5" (path "/6a022b51-582b-478a-88ab-528b7c0cb8e3/cdfcfd2c-3c7a-4183-aa6d-700ec5c19d6e" (reference "#PWR5032018") (unit 1)))))
 (wire (pts (xy 30.48 58.42) (xy 38.1 58.42)) (stroke (width 0) (type default)))
 (wire (pts (xy 38.1 58.42) (xy 55.88 58.42)) (stroke (width 0) (type default)))
@@
 (wire (pts (xy 335.28 200.66) (xy 335.28 203.2)) (stroke (width 0) (type default)))
 (wire (pts (xy 370.84 119.38) (xy 370.84 121.92)) (stroke (width 0) (type default)))
+(wire (pts (xy 370.84 137.16) (xy 370.84 139.7)) (stroke (width 0) (type default)))
+(wire (pts (xy 370.84 154.94) (xy 370.84 157.48)) (stroke (width 0) (type default)))
 (junction (at 38.1 58.42) (diameter 0) (color 0 0 0 0))
 (junction (at 55.88 58.42) (diameter 0) (color 0 0 0 0))
@@
 (text "M.2 M-key socket" (exclude_from_sim no) (at 312.42 88.9 0) (effects (font (size 1.778 1.778) (bold yes)) (justify left top)))
 (text "3.33 V from VFB 0.6 V" (exclude_from_sim no) (at 137.16 101.6 0) (effects (font (size 1.27 1.27)) (justify left top)))
-(text "PCIE_PWR_EN switches the socket supply; R703 keeps it off until the CM5 drives it.\nLane 0 runs at spec polarity; H701 is the drive standoff." (exclude_from_sim no) (at 25.4 254 0) (effects (font (size 1.27 1.27)) (justify left top)))
+(text "PCIE_PWR_EN switches the socket supply; R703 keeps it off until the CM5 drives it.\nLane 0 runs at spec polarity; standoffs H701, H702 and H703 take 2280, 2230 and 2242 drives." (exclude_from_sim no) (at 25.4 254 0) (effects (font (size 1.27 1.27)) (justify left top)))
 (embedded_fonts no)
 )
