File: hardware/boards/cm5/cm5.kicad_sch (KiCad schematic)
At the start: 0 parts

Commit message: feat(hardware): use stocked CM5 headers
Other:
- note added: "Header to the main board, SIDE_BUS feed"
- note added: "Raspberry Pi CM5 host for the main board"
- note removed: "Flex to the main board, SIDE_BUS feed"
- note removed: "Raspberry Pi CM5 host for the main board, joined by the side-link flex"
Changed lines of the file:
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@@
 (text "CM5 connectors, 5 V input, fan" (exclude_from_sim no) (at 30.48 67.31 0) (effects (font (size 1.27 1.27)) (justify left top)))
 (text "Main-board link and power" (exclude_from_sim no) (at 25.4 96.52 0) (effects (font (size 1.778 1.778) (bold yes)) (justify left top)))
-(text "Flex to the main board, SIDE_BUS feed" (exclude_from_sim no) (at 30.48 118.11 0) (effects (font (size 1.27 1.27)) (justify left top)))
+(text "Header to the main board, SIDE_BUS feed" (exclude_from_sim no) (at 30.48 118.11 0) (effects (font (size 1.27 1.27)) (justify left top)))
 (text "SIDE_BUS to 5 V, 8 A buck" (exclude_from_sim no) (at 157.48 118.11 0) (effects (font (size 1.27 1.27)) (justify left top)))
 (text "External ports" (exclude_from_sim no) (at 25.4 147.32 0) (effects (font (size 1.778 1.778) (bold yes)) (justify left top)))
@@
 (text "M.2 M-key socket and 3.3 V supply" (exclude_from_sim no) (at 30.48 219.71 0) (effects (font (size 1.27 1.27)) (justify left top)))
 (text "IASIS CM5 — side board" (exclude_from_sim no) (at 25.4 20.32 0) (effects (font (size 2.54 2.54) (bold yes)) (justify left top)))
-(text "Raspberry Pi CM5 host for the main board, joined by the side-link flex" (exclude_from_sim no) (at 25.4 26.67 0) (effects (font (size 1.27 1.27)) (justify left top)))
+(text "Raspberry Pi CM5 host for the main board" (exclude_from_sim no) (at 25.4 26.67 0) (effects (font (size 1.27 1.27)) (justify left top)))
 (sheet
 		(at 25.4 55.88)
